Commit message: разобрал файлы описания робота

File: four_ws_robot_description/urdf/base/base.gazebo.xacro (robot description, xacro)
@@ -1,10 +1,10 @@
 <?xml version="1.0"?>
 <robot xmlns:xacro="http://ros.org/wiki/xacro">
-  <xacro:macro name="base_gazebo_v0">
-	<gazebo reference="base_link">
-	  <selfCollide>false</selfCollide>
-      <mu1 value="0.05" />
-      <mu2 value="0.05" />
-    </gazebo>
-  </xacro:macro>
+    <xacro:macro name="base_gazebo_v0">
+        <gazebo reference="base_link">
+            <selfCollide>false</selfCollide>
+            <mu1 value="0.05" />
+            <mu2 value="0.05" />
+        </gazebo>
+    </xacro:macro>
 </robot>

File: four_ws_robot_description/urdf/base/base.urdf.xacro (robot description, xacro)
@@ -1,28 +1,28 @@
 <?xml version="1.0"?>
 <robot xmlns:xacro="http://ros.org/wiki/xacro">
-  <xacro:include filename="$(find four_ws_robot_description)/urdf/base/base.gazebo.xacro"/>
-  <xacro:macro name="base_v0" params="parent *joint_origin">
-	<joint name="base_link_joint" type="fixed">
-	  <xacro:insert_block name="joint_origin"/>
-	  <parent link="${parent}"/>
-	  <child link="base_link"/>
-	</joint>
-	<link name="base_link">
-	  <visual>
-		<geometry>
-		  <mesh filename="package://four_ws_robot_description/meshes/DAE/base/base_link.dae"/>
-		</geometry>
-	  </visual>
-	  <collision>
-		<geometry>
-		  <mesh filename="package://four_ws_robot_description/meshes/STL/base/base_link.stl"/>
-		</geometry>
-	  </collision>
-	  <inertial>
-		<origin xyz="0 0 0.017"/>
-		<mass value="1.2"/>
-		<inertia ixx="0.0001873" ixy="0" ixz="0" iyy="0.000055" iyz="0" izz="0.0002283" />
-	  </inertial>
-	</link>
-  </xacro:macro>
+    <xacro:include filename="$(find four_ws_robot_description)/urdf/base/base.gazebo.xacro" />
+    <xacro:macro name="base_v0" params="parent *joint_origin">
+        <joint name="base_link_joint" type="fixed">
+            <xacro:insert_block name="joint_origin" />
+            <parent link="${parent}" />
+            <child link="base_link" />
+        </joint>
+        <link name="base_link">
+            <visual>
+                <geometry>
+                    <mesh filename="package://four_ws_robot_description/meshes/DAE/base/base_link.dae" />
+                </geometry>
+            </visual>
+            <collision>
+                <geometry>
+                    <mesh filename="package://four_ws_robot_description/meshes/STL/base/base_link.stl" />
+                </geometry>
+            </collision>
+            <inertial>
+                <origin xyz="0 0 0.017" />
+                <mass value="1.2" />
+                <inertia ixx="0.0001873" ixy="0" ixz="0" iyy="0.000055" iyz="0" izz="0.0002283" />
+            </inertial>
+        </link>
+    </xacro:macro>
 </robot>

File: four_ws_robot_description/urdf/lidar_base/lidar_base.gazebo.xacro (robot description, xacro)
@@ -1,10 +1,10 @@
 <?xml version="1.0"?>
 <robot xmlns:xacro="http://ros.org/wiki/xacro">
-  <xacro:macro name="lidar_base_gazebo_v0">
-	<gazebo reference="lidar_base_link">
-	  <selfCollide>false</selfCollide>
-      <mu1 value="0.05" />
-      <mu2 value="0.05" />
-    </gazebo>
-  </xacro:macro>
+    <xacro:macro name="lidar_base_gazebo_v0">
+        <gazebo reference="lidar_base_link">
+            <selfCollide>false</selfCollide>
+            <mu1 value="0.05" />
+            <mu2 value="0.05" />
+        </gazebo>
+    </xacro:macro>
 </robot>

File: four_ws_robot_description/urdf/lidar_base/lidar_base.urdf.xacro (robot description, xacro)
@@ -1,28 +1,28 @@
 <?xml version="1.0"?>
 <robot xmlns:xacro="http://ros.org/wiki/xacro">
-  <xacro:include filename="$(find four_ws_robot_description)/urdf/lidar_base/lidar_base.gazebo.xacro"/>
-  <xacro:macro name="lidar_base_v0" params="parent *joint_origin">
-	<joint name="lidar_base_link_joint" type="fixed">
-	  <xacro:insert_block name="joint_origin"/>
-	  <parent link="${parent}"/>
-	  <child link="lidar_base_link"/>
-	</joint>
-	<link name="lidar_base_link">
-	  <visual>
-		<geometry>
-		  <mesh filename="package://four_ws_robot_description/meshes/DAE/lidar_base/YDlidar_base.dae"/>
-		</geometry>
-	  </visual>
-	  <collision>
-		<geometry>
-		  <mesh filename="package://four_ws_robot_description/meshes/STL/lidar_base/YDlidar_base.stl"/>
-		</geometry>
-	  </collision>
-	  <inertial>
-		<origin xyz="0 0 0.017"/>
-		<mass value="0.2"/>
-		<inertia ixx="0.0000873" ixy="0" ixz="0" iyy="0.000005" iyz="0" izz="0.0000283" />
-	  </inertial>
-	</link>
-  </xacro:macro>
+    <xacro:include filename="$(find four_ws_robot_description)/urdf/lidar_base/lidar_base.gazebo.xacro" />
+    <xacro:macro name="lidar_base_v0" params="parent *joint_origin">
+        <joint name="lidar_base_link_joint" type="fixed">
+            <xacro:insert_block name="joint_origin" />
+            <parent link="${parent}" />
+            <child link="lidar_base_link" />
+        </joint>
+        <link name="lidar_base_link">
+            <visual>
+                <geometry>
+                    <mesh filename="package://four_ws_robot_description/meshes/DAE/lidar_base/YDlidar_base.dae" />
+                </geometry>
+            </visual>
+            <collision>
+                <geometry>
+                    <mesh filename="package://four_ws_robot_description/meshes/STL/lidar_base/YDlidar_base.stl" />
+                </geometry>
+            </collision>
+            <inertial>
+                <origin xyz="0 0 0.017" />
+                <mass value="0.2" />
+                <inertia ixx="0.0000873" ixy="0" ixz="0" iyy="0.000005" iyz="0" izz="0.0000283" />
+            </inertial>
+        </link>
+    </xacro:macro>
 </robot>

File: four_ws_robot_description/urdf/lidar_head/lidar_head.gazebo.xacro (robot description, xacro)
@@ -1,10 +1,10 @@
 <?xml version="1.0"?>
 <robot xmlns:xacro="http://ros.org/wiki/xacro">
-  <xacro:macro name="lidar_head_gazebo_v0">
-    <gazebo reference="lidar_head_link">
-      <selfCollide>false</selfCollide>
-      <mu1 value="0.05" />
-      <mu2 value="0.05" />
-    </gazebo>
-  </xacro:macro>
+    <xacro:macro name="lidar_head_gazebo_v0">
+        <gazebo reference="lidar_head_link">
+            <selfCollide>false</selfCollide>
+            <mu1 value="0.05" />
+            <mu2 value="0.05" />
+        </gazebo>
+    </xacro:macro>
 </robot>

File: four_ws_robot_description/urdf/lidar_head/lidar_head.transmission.xacro (robot description, xacro)
@@ -1,15 +1,15 @@
 <?xml version="1.0"?>
 <robot xmlns:xacro="http://ros.org/wiki/xacro">
-  <xacro:macro name="lidar_trans_v0">
-    <transmission name="lidar_head_trans">
-      <type>transmission_interface/SimpleTransmission</type>
-      <joint name="lidar_head_joint">
-	<hardwareInterface>hardware_interface/VelocityJointInterface</hardwareInterface>
-      </joint>
-	<actuator name="lidar_head_motor">
-	  <hardwareInterface>hardware_interface/VelocityJointInterface</hardwareInterface>
-	  <mechanicalReduction>1</mechanicalReduction>
-        </actuator>
-    </transmission>
-  </xacro:macro>
+    <xacro:macro name="lidar_trans_v0">
+        <transmission name="lidar_head_trans">
+            <type>transmission_interface/SimpleTransmission</type>
+            <joint name="lidar_head_joint">
+                <hardwareInterface>hardware_interface/VelocityJointInterface</hardwareInterface>
+            </joint>
+            <actuator name="lidar_head_motor">
+                <hardwareInterface>hardware_interface/VelocityJointInterface</hardwareInterface>
+                <mechanicalReduction>1</mechanicalReduction>
+            </actuator>
+        </transmission>
+    </xacro:macro>
 </robot>

File: four_ws_robot_description/urdf/lidar_head/lidar_head.urdf.xacro (robot description, xacro)
@@ -1,31 +1,31 @@
 <?xml version="1.0"?>
 <robot xmlns:xacro="http://ros.org/wiki/xacro">
-  <xacro:include filename="$(find four_ws_robot_description)/urdf/lidar_head/lidar_head.transmission.xacro"/>
-  <xacro:include filename="$(find four_ws_robot_description)/urdf/lidar_head/lidar_head.gazebo.xacro"/>
-  <xacro:macro name="lidar_head_v0" params="parent *joint_origin *joint_axis">
-	<joint name="lidar_head_joint" type="continuous">
-	  <xacro:insert_block name="joint_origin"/>
-	  <parent link="${parent}"/>
-	  <child link="lidar_head_link"/>
-         <limit effort="1.5" velocity="20"/>
-	  <xacro:insert_block name="joint_axis"/>
-	</joint>
-	<link name="lidar_head_link">
-	  <visual>
-		<geometry>
-		  <mesh filename="package://four_ws_robot_description/meshes/DAE/lidar_head/YDlidar_head.dae"/>
-		</geometry>
-	  </visual>
-	  <collision>
-		<geometry>
-		  <mesh filename="package://four_ws_robot_description/meshes/STL/lidar_head/YDlidar_head.stl"/>
-		</geometry>
-	  </collision>
-	  <inertial>
-		<origin xyz="0.0 0 0"/>
-		<mass value="0.05"/>
-		<inertia ixx="0.00001" ixy="0" ixz="0" iyy="0.000018" iyz="0" izz="0.00001"/>
-	  </inertial>
-	</link>
-  </xacro:macro>
+    <xacro:include filename="$(find four_ws_robot_description)/urdf/lidar_head/lidar_head.transmission.xacro" />
+    <xacro:include filename="$(find four_ws_robot_description)/urdf/lidar_head/lidar_head.gazebo.xacro" />
+    <xacro:macro name="lidar_head_v0" params="parent *joint_origin *joint_axis">
+        <joint name="lidar_head_joint" type="continuous">
+            <xacro:insert_block name="joint_origin" />
+            <parent link="${parent}" />
+            <child link="lidar_head_link" />
+            <limit effort="1.5" velocity="20" />
+            <xacro:insert_block name="joint_axis" />
+        </joint>
+        <link name="lidar_head_link">
+            <visual>
+                <geometry>
+                    <mesh filename="package://four_ws_robot_description/meshes/DAE/lidar_head/YDlidar_head.dae" />
+                </geometry>
+            </visual>
+            <collision>
+                <geometry>
+                    <mesh filename="package://four_ws_robot_description/meshes/STL/lidar_head/YDlidar_head.stl" />
+                </geometry>
+            </collision>
+            <inertial>
+                <origin xyz="0.0 0 0" />
+                <mass value="0.05" />
+                <inertia ixx="0.00001" ixy="0" ixz="0" iyy="0.000018" iyz="0" izz="0.00001" />
+            </inertial>
+        </link>
+    </xacro:macro>
 </robot>

File: four_ws_robot_description/urdf/lrf/lrf.gazebo.xacro (robot description, xacro)
@@ -1,36 +1,37 @@
 <?xml version="1.0"?>
 <robot xmlns:xacro="http://ros.org/wiki/xacro">
-  <xacro:macro name="lrf_gazebo_v0" params="prefix min_rad max_rad min_range max_range">
-	<gazebo reference="${prefix}_lrf_link">
-      <sensor type="ray" name="${prefix}_lrf_sensor">
-		<pose>0 0 0 0 0 0</pose>
-		<visualize>true</visualize>
-		<update_rate>40</update_rate>
-		<ray>
-          <scan>
-	    <horizontal>
-              <samples>720</samples>
-              <resolution>1</resolution>
-              <min_angle>${min_rad}</min_angle>
-              <max_angle>${max_rad}</max_angle>
-	    </horizontal>
-          </scan>
-          <range>
-		<min>${min_range}</min>
-		<max>${max_range}</max>
-		<resolution>0.01</resolution>
-          </range>
-          <noise>
-		<type>gaussian</type>
-		<mean>0.0</mean>
-		<stddev>0.03</stddev>
-          </noise>
-		</ray>
-		<plugin name="gazebo_ros_${prefix}_lrf_controller" filename="libgazebo_ros_laser.so">
-          <topicName>${prefix}/scan</topicName> <!-- do ont set it to base_scan -->
-          <frameName>${prefix}_lrf_link</frameName>
-		</plugin>
-      </sensor>
-	</gazebo>
-  </xacro:macro>
+    <xacro:macro name="lrf_gazebo_v0" params="prefix min_rad max_rad min_range max_range">
+        <gazebo reference="${prefix}_lrf_link">
+            <sensor type="ray" name="${prefix}_lrf_sensor">
+                <pose>0 0 0 0 0 0</pose>
+                <visualize>true</visualize>
+                <update_rate>40</update_rate>
+                <ray>
+                    <scan>
+                        <horizontal>
+                            <samples>720</samples>
+                            <resolution>1</resolution>
+                            <min_angle>${min_rad}</min_angle>
+                            <max_angle>${max_rad}</max_angle>
+                        </horizontal>
+                    </scan>
+                    <range>
+                        <min>${min_range}</min>
+                        <max>${max_range}</max>
+                        <resolution>0.01</resolution>
+                    </range>
+                    <noise>
+                        <type>gaussian</type>
+                        <mean>0.0</mean>
+                        <stddev>0.03</stddev>
+                    </noise>
+                </ray>
+                <plugin name="gazebo_ros_${prefix}_lrf_controller" filename="libgazebo_ros_laser.so">
+                    <topicName>${prefix}/scan</topicName>
+                    <!-- do ont set it to base_scan -->
+                    <frameName>${prefix}_lrf_link</frameName>
+                </plugin>
+            </sensor>
+        </gazebo>
+    </xacro:macro>
 </robot>

File: four_ws_robot_description/urdf/lrf/lrf.urdf.xacro (robot description, xacro)
@@ -1,13 +1,12 @@
 <?xml version="1.0"?>
 <robot xmlns:xacro="http://ros.org/wiki/xacro">
-  <xacro:include filename="$(find four_ws_robot_description)/urdf/lrf/lrf.gazebo.xacro"/>
-  <xacro:macro name="lrf_v0" params="prefix parent *joint_origin">
-	<joint name="${prefix}_lrf_joint" type="fixed">
-	  <xacro:insert_block name="joint_origin"/>
-	  <parent link="${parent}"/>
-	  <child link="${prefix}_lrf_link"/>
-	</joint>
-	<link name="${prefix}_lrf_link">
-	</link>
-  </xacro:macro>
+    <xacro:include filename="$(find four_ws_robot_description)/urdf/lrf/lrf.gazebo.xacro" />
+    <xacro:macro name="lrf_v0" params="prefix parent *joint_origin">
+        <joint name="${prefix}_lrf_joint" type="fixed">
+            <xacro:insert_block name="joint_origin" />
+            <parent link="${parent}" />
+            <child link="${prefix}_lrf_link" />
+        </joint>
+        <link name="${prefix}_lrf_link" />
+    </xacro:macro>
 </robot>

File: four_ws_robot_description/urdf/suspension/suspension.gazebo.xacro (robot description, xacro)
@@ -1,10 +1,14 @@
 <?xml version="1.0"?>
+<!-- Файл "suspension.gazebo.xacro" описывает параметры модели подвески робота для симуляции
+в среде Gazebo. Он содержит макрос "steering_gazebo_v0", который определяет параметры для
+элемента "gazebo" в модели, такие как самостолкновение, коэффициенты трения между
+элементами модели и другие параметры. -->
 <robot xmlns:xacro="http://ros.org/wiki/xacro">
-  <xacro:macro name="steering_gazebo_v0" params="prefix">
-	<gazebo reference="${prefix}_steering_link">
-	  <selfCollide>false</selfCollide>
-      <mu1 value="0.05" />
-      <mu2 value="0.05" />
-    </gazebo>
-  </xacro:macro>
+    <xacro:macro name="steering_gazebo_v0" params="prefix">
+        <gazebo reference="${prefix}_steering_link">
+            <selfCollide>false</selfCollide>
+            <mu1 value="0.05" />
+            <mu2 value="0.05" />
+        </gazebo>
+    </xacro:macro>
 </robot>

File: four_ws_robot_description/urdf/suspension/suspension.transmission.xacro (robot description, xacro)
@@ -1,15 +1,20 @@
 <?xml version="1.0"?>
+<!-- Файл "suspension.transmission.xacro" определяет параметры трансмиссии робота.
+Он содержит макрос "steering_trans_v0", который определяет параметры трансмиссии,
+такие как тип трансмиссии (в данном случае "transmission_interface/SimpleTransmission"),
+аппаратный интерфейс для соединения с мотором и суставом, а также
+механическое уменьшение (mechanicalReduction) для мотора. -->
 <robot xmlns:xacro="http://ros.org/wiki/xacro">
-  <xacro:macro name="steering_trans_v0" params="prefix">
-	<transmission name="${prefix}_steering_trans">
-      <type>transmission_interface/SimpleTransmission</type>
-      <joint name="${prefix}_steering_joint">
-		<hardwareInterface>hardware_interface/PositionJointInterface</hardwareInterface>
-      </joint>
-	  <actuator name="${prefix}_steering_motor">
-		<hardwareInterface>hardware_interface/PositionJointInterface</hardwareInterface>
-		<mechanicalReduction>30</mechanicalReduction>
-      </actuator>
-	</transmission>
-  </xacro:macro>
+    <xacro:macro name="steering_trans_v0" params="prefix">
+        <transmission name="${prefix}_steering_trans">
+            <type>transmission_interface/SimpleTransmission</type>
+            <joint name="${prefix}_steering_joint">
+                <hardwareInterface>hardware_interface/PositionJointInterface</hardwareInterface>
+            </joint>
+            <actuator name="${prefix}_steering_motor">
+                <hardwareInterface>hardware_interface/PositionJointInterface</hardwareInterface>
+                <mechanicalReduction>30</mechanicalReduction>
+            </actuator>
+        </transmission>
+    </xacro:macro>
 </robot>

File: four_ws_robot_description/urdf/suspension/suspension.urdf.xacro (robot description, xacro)
@@ -1,31 +1,36 @@
 <?xml version="1.0"?>
+<!-- Файл "suspension.urdf.xacro" объединяет описания подвески робота,
+используя включения (include), и определяет макрос "steering_v0", который
+определяет параметры соединения сустава робота. Он содержит описание соединения
+сустава, такие как тип соединения (revolute), ограничения на усилие, скорость и
+ограничения на угол поворота сустава, а также геометрию визуализации и коллизий сустава. -->
 <robot xmlns:xacro="http://ros.org/wiki/xacro">
-  <xacro:include filename="$(find four_ws_robot_description)/urdf/suspension/suspension.transmission.xacro"/>
-  <xacro:include filename="$(find four_ws_robot_description)/urdf/suspension/suspension.gazebo.xacro"/>
-  <xacro:macro name="steering_v0" params="prefix parent *joint_origin *joint_axis">
-	<joint name="${prefix}_steering_joint" type="revolute">
-	  <xacro:insert_block name="joint_origin"/>
-	  <parent link="${parent}"/>
-	  <child link="${prefix}_steering_link"/>
-          <limit effort="5" velocity="6.28"  lower="-2.1" upper="2.1" />
-          <xacro:insert_block name="joint_axis"/>
-	</joint>
-	<link name="${prefix}_steering_link">
-	  <visual>
-		<geometry>
-		  <mesh filename="package://four_ws_robot_description/meshes/DAE/suspension/${prefix}_link.dae"/>
-		</geometry>
-	  </visual>
-	  <collision>
-		<geometry>
-		  <mesh filename="package://four_ws_robot_description/meshes/STL/suspension/sus_link.stl"/>
-		</geometry>
-	  </collision>
-	  <inertial>
-		<origin xyz="0 0 -0.02"/>
-		<mass value="0.15"/>
-		<inertia ixx="0.00001" ixy="0" ixz="0" iyy="0.00001" iyz="0" izz="0.000004" />
-	  </inertial>
-	</link>
-  </xacro:macro>
+    <xacro:include filename="$(find four_ws_robot_description)/urdf/suspension/suspension.transmission.xacro" />
+    <xacro:include filename="$(find four_ws_robot_description)/urdf/suspension/suspension.gazebo.xacro" />
+    <xacro:macro name="steering_v0" params="prefix parent *joint_origin *joint_axis">
+        <joint name="${prefix}_steering_joint" type="revolute">
+            <xacro:insert_block name="joint_origin" />
+            <parent link="${parent}" />
+            <child link="${prefix}_steering_link" />
+            <limit effort="5" velocity="6.28" lower="-2.1" upper="2.1" />
+            <xacro:insert_block name="joint_axis" />
+        </joint>
+        <link name="${prefix}_steering_link">
+            <visual>
+                <geometry>
+                    <mesh filename="package://four_ws_robot_description/meshes/DAE/suspension/${prefix}_link.dae" />
+                </geometry>
+            </visual>
+            <collision>
+                <geometry>
+                    <mesh filename="package://four_ws_robot_description/meshes/STL/suspension/sus_link.stl" />
+                </geometry>
+            </collision>
+            <inertial>
+                <origin xyz="0 0 -0.02" />
+                <mass value="0.15" />
+                <inertia ixx="0.00001" ixy="0" ixz="0" iyy="0.00001" iyz="0" izz="0.000004" />
+            </inertial>
+        </link>
+    </xacro:macro>
 </robot>

File: four_ws_robot_description/urdf/wheel/wheel.gazebo.xacro (robot description, xacro)
@@ -1,10 +1,15 @@
 <?xml version="1.0"?>
+<!-- Файл wheel.gazebo.xacro содержит описание модели колеса для симулятора Gazebo.
+Внутри макроса wheel_gazebo_v0 определены параметры, такие как ссылка на соответствующее
+звено колеса в URDF модели (${prefix}_wheel_link) и коэффициенты трения mu1 и mu2,
+установленные в значения 1.2. Значения коэффициентов трения mu1 и mu2 определяют трение
+между колесом и поверхностью, где робот будет симулирован в среде Gazebo. -->
 <robot xmlns:xacro="http://ros.org/wiki/xacro">
-  <xacro:macro name="wheel_gazebo_v0" params="prefix">
-    <gazebo reference="${prefix}_wheel_link">
-      <selfCollide>false</selfCollide>
-      <mu1 value="1.2" />
-      <mu2 value="1.2" />
-    </gazebo>
-  </xacro:macro>
+    <xacro:macro name="wheel_gazebo_v0" params="prefix">
+        <gazebo reference="${prefix}_wheel_link">
+            <selfCollide>false</selfCollide>
+            <mu1 value="1.2" />
+            <mu2 value="1.2" />
+        </gazebo>
+    </xacro:macro>
 </robot>

File: four_ws_robot_description/urdf/wheel/wheel.transmission.xacro (robot description, xacro)
@@ -1,15 +1,21 @@
 <?xml version="1.0"?>
+<!-- Файл wheel.transmission.xacro содержит описание трансмиссии (передачи) для колеса робота.
+Внутри макроса wheel_trans_v0 определены параметры, такие как название трансмиссии
+(${prefix}_wheel_trans), тип трансмиссии (transmission_interface/SimpleTransmission),
+а также интерфейсы обмена данными с аппаратным обеспечением
+(hardware_interface/VelocityJointInterface) для соединения колеса
+с мотором иуправления его скоростью. -->
 <robot xmlns:xacro="http://ros.org/wiki/xacro">
-  <xacro:macro name="wheel_trans_v0" params="prefix">
-    <transmission name="${prefix}_wheel_trans">
-      <type>transmission_interface/SimpleTransmission</type>
-      <joint name="${prefix}_wheel_joint">
-	<hardwareInterface>hardware_interface/VelocityJointInterface</hardwareInterface>
-      </joint>
-	<actuator name="${prefix}_wheel_motor">
-	  <hardwareInterface>hardware_interface/VelocityJointInterface</hardwareInterface>
-	  <mechanicalReduction>1</mechanicalReduction>
-        </actuator>
-    </transmission>
-  </xacro:macro>
+    <xacro:macro name="wheel_trans_v0" params="prefix">
+        <transmission name="${prefix}_wheel_trans">
+            <type>transmission_interface/SimpleTransmission</type>
+            <joint name="${prefix}_wheel_joint">
+                <hardwareInterface>hardware_interface/VelocityJointInterface</hardwareInterface>
+            </joint>
+            <actuator name="${prefix}_wheel_motor">
+                <hardwareInterface>hardware_interface/VelocityJointInterface</hardwareInterface>
+                <mechanicalReduction>1</mechanicalReduction>
+            </actuator>
+        </transmission>
+    </xacro:macro>
 </robot>
