Commit message: привел файлы описания деталей робота к стандартному виду + заменил модель столкновения (предыдушая версия была повернута на 90 гр) + убрал ПИД для лидара потому что его все равно колбасит + в добавил требуемый пакет

File: four_ws_robot_description/urdf/base/base.urdf.xacro (robot description, xacro)
@@ -13,4 +13,5 @@
                     <mesh filename="package://four_ws_robot_description/meshes/DAE/base/base_link.dae" />
                 </geometry>
+                <origin xyz="0.0 0.0 0.0" />
             </visual>
             <collision>
@@ -18,8 +19,9 @@
                     <mesh filename="package://four_ws_robot_description/meshes/STL/base/base_link.stl" />
                 </geometry>
+                <origin xyz="0.0 0.0 0.0" />
             </collision>
             <inertial>
+                <mass value="1.2" />
                 <origin xyz="0 0 0.017" />
-                <mass value="1.2" />
                 <inertia ixx="0.0001873" ixy="0" ixz="0" iyy="0.000055" iyz="0" izz="0.0002283" />
             </inertial>

File: four_ws_robot_description/urdf/lidar_base/lidar_base.urdf.xacro (robot description, xacro)
@@ -13,4 +13,5 @@
                     <mesh filename="package://four_ws_robot_description/meshes/DAE/lidar_base/YDlidar_base.dae" />
                 </geometry>
+                <origin xyz="0.0 0.0 0.0" />
             </visual>
             <collision>
@@ -18,8 +19,9 @@
                     <mesh filename="package://four_ws_robot_description/meshes/STL/lidar_base/YDlidar_base.stl" />
                 </geometry>
+                <origin xyz="0.0 0.0 0.0" />
             </collision>
             <inertial>
-                <origin xyz="0 0 0.017" />
                 <mass value="0.2" />
+                <origin xyz="0.0 0.0 0.017" />
                 <inertia ixx="0.0000873" ixy="0" ixz="0" iyy="0.000005" iyz="0" izz="0.0000283" />
             </inertial>

File: four_ws_robot_description/urdf/lidar_head/lidar_head.urdf.xacro (robot description, xacro)
@@ -16,4 +16,5 @@
                     <mesh filename="package://four_ws_robot_description/meshes/DAE/lidar_head/YDlidar_head.dae" />
                 </geometry>
+                <origin xyz="0.0 0.0 0.0" />
             </visual>
             <collision>
@@ -21,8 +22,9 @@
                     <mesh filename="package://four_ws_robot_description/meshes/STL/lidar_head/YDlidar_head.stl" />
                 </geometry>
+                <origin xyz="0.0 0.0 0.0" />
             </collision>
             <inertial>
-                <origin xyz="0.0 0 0" />
                 <mass value="0.05" />
+                <origin xyz="0.0 0.0 0.0" />
                 <inertia ixx="0.00001" ixy="0" ixz="0" iyy="0.000018" iyz="0" izz="0.00001" />
             </inertial>

File: four_ws_robot_description/urdf/suspension/suspension.gazebo.xacro (robot description, xacro)
@@ -1,7 +1,3 @@
 <?xml version="1.0"?>
-<!-- Файл "suspension.gazebo.xacro" описывает параметры модели подвески робота для симуляции
-в среде Gazebo. Он содержит макрос "steering_gazebo", который определяет параметры для
-элемента "gazebo" в модели, такие как самостолкновение, коэффициенты трения между
-элементами модели и другие параметры. -->
 <robot xmlns:xacro="http://ros.org/wiki/xacro">
     <xacro:macro name="steering_gazebo" params="prefix">

File: four_ws_robot_description/urdf/suspension/suspension.transmission.xacro (robot description, xacro)
@@ -1,8 +1,3 @@
 <?xml version="1.0"?>
-<!-- Файл "suspension.transmission.xacro" определяет параметры трансмиссии робота.
-Он содержит макрос "steering_trans", который определяет параметры трансмиссии,
-такие как тип трансмиссии (в данном случае "transmission_interface/SimpleTransmission"),
-аппаратный интерфейс для соединения с мотором и суставом, а также
-механическое уменьшение (mechanicalReduction) для мотора. -->
 <robot xmlns:xacro="http://ros.org/wiki/xacro">
     <xacro:macro name="steering_trans" params="prefix">

File: four_ws_robot_description/urdf/suspension/suspension.urdf.xacro (robot description, xacro)
@@ -1,8 +1,3 @@
 <?xml version="1.0"?>
-<!-- Файл "suspension.urdf.xacro" объединяет описания подвески робота,
-используя включения (include), и определяет макрос "steering", который
-определяет параметры соединения сустава робота. Он содержит описание соединения
-сустава, такие как тип соединения (revolute), ограничения на усилие, скорость и
-ограничения на угол поворота сустава, а также геометрию визуализации и коллизий сустава. -->
 <robot xmlns:xacro="http://ros.org/wiki/xacro">
     <xacro:include filename="$(find four_ws_robot_description)/urdf/suspension/suspension.transmission.xacro" />
@@ -21,4 +16,5 @@
                     <mesh filename="package://four_ws_robot_description/meshes/DAE/suspension/${prefix}_link.dae" />
                 </geometry>
+                <origin xyz="0.0 0.0 0.0" />
             </visual>
             <collision>
@@ -26,8 +22,9 @@
                     <mesh filename="package://four_ws_robot_description/meshes/STL/suspension/sus_link.stl" />
                 </geometry>
+                <origin xyz="0.0 0.0 0.0" />
             </collision>
             <inertial>
-                <origin xyz="0 0 -0.02" />
                 <mass value="0.15" />
+                <origin xyz="0.0 0.0 -0.02" />
                 <inertia ixx="0.00001" ixy="0" ixz="0" iyy="0.00001" iyz="0" izz="0.000004" />
             </inertial>

File: four_ws_robot_description/urdf/wheel/wheel.gazebo.xacro (robot description, xacro)
@@ -1,8 +1,3 @@
 <?xml version="1.0"?>
-<!-- Файл wheel.gazebo.xacro содержит описание модели колеса для симулятора Gazebo.
-Внутри макроса wheel_gazebo определены параметры, такие как ссылка на соответствующее
-звено колеса в URDF модели (${prefix}_wheel_link) и коэффициенты трения mu1 и mu2,
-установленные в значения 1.2. Значения коэффициентов трения mu1 и mu2 определяют трение
-между колесом и поверхностью, где робот будет симулирован в среде Gazebo. -->
 <robot xmlns:xacro="http://ros.org/wiki/xacro">
     <xacro:macro name="wheel_gazebo" params="prefix">

File: four_ws_robot_description/urdf/wheel/wheel.transmission.xacro (robot description, xacro)
@@ -1,9 +1,3 @@
 <?xml version="1.0"?>
-<!-- Файл wheel.transmission.xacro содержит описание трансмиссии (передачи) для колеса робота.
-Внутри макроса wheel_trans определены параметры, такие как название трансмиссии
-(${prefix}_wheel_trans), тип трансмиссии (transmission_interface/SimpleTransmission),
-а также интерфейсы обмена данными с аппаратным обеспечением
-(hardware_interface/VelocityJointInterface) для соединения колеса
-с мотором иуправления его скоростью. -->
 <robot xmlns:xacro="http://ros.org/wiki/xacro">
     <xacro:macro name="wheel_trans" params="prefix">

File: four_ws_robot_description/urdf/wheel/wheel.urdf.xacro (robot description, xacro)
@@ -1,10 +1,3 @@
 <?xml version="1.0"?>
-<!-- Файл wheel.urdf.xacro содержит полное описание колеса робота в формате URDF
-(Unified Robot Description Format), который используется для описания геометрии,
-кинематики, инерционных свойств и других характеристик робота.
-Внутри макроса wheel определены параметры, такие как название звена колеса
-(${prefix}_wheel_link), тип и ограничения соединения (<joint>),
-геометрия визуализации и столкновений колеса (<visual> и <collision>),
-а также инерционные свойства (<inertial>) для симуляции физических характеристик колеса. -->
 <robot xmlns:xacro="http://ros.org/wiki/xacro">
     <xacro:include filename="$(find four_ws_robot_description)/urdf/wheel/wheel.transmission.xacro" />
@@ -23,4 +16,5 @@
                     <mesh filename="package://four_ws_robot_description/meshes/DAE/wheel/wheel_link.dae" />
                 </geometry>
+                <origin xyz="0.0 0.0 0.0" />
             </visual>
             <collision>
@@ -28,8 +22,9 @@
                     <mesh filename="package://four_ws_robot_description/meshes/STL/wheel/robot_wheel.stl" />
                 </geometry>
+                <origin xyz="0.0 0.0 0.0" />
             </collision>
             <inertial>
-                <origin xyz="0.0 -0.007 -0.0" />
                 <mass value="0.05" />
+                <origin xyz="0.0 -0.007 0.0" />
                 <inertia ixx="0.00001" ixy="0" ixz="0" iyy="0.000018" iyz="0" izz="0.00001" />
             </inertial>
