Commit message: убрал модели неиспользуемых сенсоров

File: four_ws_robot_description/urdf/camera/camera.urdf.xacro (robot description, xacro)
@@ -10,5 +10,5 @@
             <visual>
                 <geometry>
-                    <mesh filename="package://four_ws_robot_description/meshes/DAE/camera/camera.dae" />
+                    <mesh filename="package://four_ws_robot_description/meshes/DAE/sensors/camera/camera.dae" />
                 </geometry>
                 <origin xyz="0.0 0.0 0.0" />
@@ -16,5 +16,5 @@
             <collision>
                 <geometry>
-                    <mesh filename="package://four_ws_robot_description/meshes/STL/camera/camera.stl" />
+                    <mesh filename="package://four_ws_robot_description/meshes/STL/sensors/camera/camera.stl" />
                 </geometry>
                 <origin xyz="0.0 0.0 0.0" />
