Commit message: изменены названия сочленений робота

File: four_ws_robot_description/robots/four_ws_robot.urdf.xacro (robot description, xacro)
@@ -8,22 +8,22 @@
     <xacro:include filename="$(find four_ws_robot_description)/urdf/lidar_head/lidar_head.urdf.xacro"/>
     <xacro:include filename="$(find four_ws_robot_description)/urdf/lrf/lrf.urdf.xacro"/>
-    <!-- =============== Link & Joint =============== -->
+    <!-- Link & Joint -->
     <!-- Base -->
     <link name="base_footprint"/> <!--link name="base_footprint"/ -->
     <xacro:base_v0 parent="base_footprint"> <!-- xacro:base_v0 parent="base_footprint" -->
-        <origin xyz="0 0 0"/>
+        <origin xyz="0 0 0" rpy="0 0 0"/>
     </xacro:base_v0>
     <!-- lidar_base -->
     <xacro:lidar_base_v0 parent="base_link">
-        <origin xyz="-0.022 0 0.035"/>
+        <origin xyz="-0.022 0 0.035" rpy="0 0 0"/>
     </xacro:lidar_base_v0>
     <!-- lidar_head -->
     <xacro:lidar_head_v0 parent="lidar_base_link">
-        <origin xyz="0.022 0 0.0"/>
+        <origin xyz="0.022 0 0.0" rpy="0 0 0"/>
         <axis xyz="0 0 1"/>
     </xacro:lidar_head_v0>
     <!-- lrf sensor -->
     <xacro:lrf_v0 prefix = "front" parent="base_link">
-        <origin xyz="0 0 0.083"/>
+        <origin xyz="0 0 0.083" rpy="0 0 0"/>
     </xacro:lrf_v0>
     <link name="lrf_link"/>
@@ -31,58 +31,58 @@
         <parent link="base_link"/>
         <child link="lrf_link"/>
-        <origin xyz="0 0 0.01"/>
+        <origin xyz="0 0 0.01" rpy="0 0 0"/>
     </joint>
     <!-- Suspension -->
     <!-- Front Right Sus -->
     <xacro:steering_v0 prefix="front_right" parent="base_link">
-        <origin xyz="0.077 -0.031 -0.004"/>
+        <origin xyz="0.077 -0.031 -0.004" rpy="0 0 0"/>
         <axis xyz="0 0 1"/>
     </xacro:steering_v0>
     <!-- Front Left Sus -->
     <xacro:steering_v0 prefix="front_left" parent="base_link">
-        <origin xyz="0.077 0.031 -0.004"/>
+        <origin xyz="0.077 0.031 -0.004" rpy="0 0 0"/>
         <axis xyz="0 0 1"/>
     </xacro:steering_v0>
     <!-- Rear Right Sus -->
     <xacro:steering_v0 prefix="rear_right" parent="base_link">
-        <origin xyz="-0.077 -0.031 -0.004"/>
+        <origin xyz="-0.077 -0.031 -0.004" rpy="0 0 0"/>
         <axis xyz="0 0 1"/>
     </xacro:steering_v0>
     <!-- Rear Left Sus -->
     <xacro:steering_v0 prefix="rear_left" parent="base_link">
-        <origin xyz="-0.077 0.031 -0.004"/>
+        <origin xyz="-0.077 0.031 -0.004" rpy="0 0 0"/>
         <axis xyz="0 0 1"/>
     </xacro:steering_v0>
     <!-- Wheel -->
+    <!-- Front Left Wheel -->
+    <xacro:wheel_v0 prefix="front_left" parent="front_left_steering_link">
+        <origin xyz="0 0.021 -0.025" rpy="0 0 ${M_PI}"/>
+        <axis xyz="0 -1 0"/>
+    </xacro:wheel_v0>
     <!-- Front Right Wheel -->
-    <xacro:wheel_v0 prefix="ffr" parent="front_right_steering_link">
-        <origin xyz="0 -0.021 -0.025"/>
+    <xacro:wheel_v0 prefix="front_right" parent="front_right_steering_link">
+        <origin xyz="0 -0.021 -0.025" rpy="0 0 0"/>
         <axis xyz="0 1 0"/>
     </xacro:wheel_v0>
-    <!--  Front Left Wheel -->
-    <xacro:wheel_v0 prefix="ffl" parent="front_left_steering_link">
+    <!--  Rear Left Wheel -->
+    <xacro:wheel_v0 prefix="rear_left" parent="rear_left_steering_link">
         <origin xyz="0 0.021 -0.025" rpy="0 0 ${M_PI}"/>
         <axis xyz="0 -1 0"/>
     </xacro:wheel_v0>
     <!-- Rear Right Wheel -->
-    <xacro:wheel_v0 prefix="rfr" parent="rear_right_steering_link">
-        <origin xyz="0 -0.021 -0.025"/>
+    <xacro:wheel_v0 prefix="rear_right" parent="rear_right_steering_link">
+        <origin xyz="0 -0.021 -0.025" rpy="0 0 0"/>
         <axis xyz="0 1 0"/>
     </xacro:wheel_v0>
-    <!--  Rear Left Wheel -->
-    <xacro:wheel_v0 prefix="rfl" parent="rear_left_steering_link">
-        <origin xyz="0 0.021 -0.025" rpy="0 0 ${M_PI}"/>
-        <axis xyz="0 -1 0"/>
-    </xacro:wheel_v0>
     <!-- ===============  Wheel Transmission =============== -->
-    <xacro:wheel_trans_v0 prefix="ffr"/>
-    <xacro:wheel_trans_v0 prefix="ffl"/>
-    <xacro:wheel_trans_v0 prefix="rfr"/>
-    <xacro:wheel_trans_v0 prefix="rfl"/>
+    <xacro:wheel_trans_v0 prefix="front_left"/>
+    <xacro:wheel_trans_v0 prefix="front_right"/>
+    <xacro:wheel_trans_v0 prefix="rear_left"/>
+    <xacro:wheel_trans_v0 prefix="rear_right"/>
     <!-- ===============  Steering Transmission =============== -->
+    <xacro:steering_trans_v0 prefix="front_left"/>
     <xacro:steering_trans_v0 prefix="front_right"/>
-    <xacro:steering_trans_v0 prefix="front_left"/>
+    <xacro:steering_trans_v0 prefix="rear_left"/>
     <xacro:steering_trans_v0 prefix="rear_right"/>
-    <xacro:steering_trans_v0 prefix="rear_left"/>
     <!-- ===============  lider head Transmission =============== -->
     <xacro:lidar_trans_v0/>
@@ -110,12 +110,12 @@
     <xacro:lrf_gazebo_v0 prefix = "front" min_rad = "-3.14" max_rad = "3.14" min_range = "0.1" max_range = "10"/>
     <!-- Wheel -->
-    <xacro:wheel_gazebo_v0 prefix="fr"/>
-    <xacro:wheel_gazebo_v0 prefix="fl"/>
-    <xacro:wheel_gazebo_v0 prefix="rr"/>
-    <xacro:wheel_gazebo_v0 prefix="rl"/>
+    <xacro:wheel_gazebo_v0 prefix="front_left"/>
+    <xacro:wheel_gazebo_v0 prefix="front_right"/>
+    <xacro:wheel_gazebo_v0 prefix="rear_left"/>
+    <xacro:wheel_gazebo_v0 prefix="rear_right"/>
     <!-- Steering -->
+    <xacro:steering_gazebo_v0 prefix="front_left"/>
     <xacro:steering_gazebo_v0 prefix="front_right"/>
-    <xacro:steering_gazebo_v0 prefix="front_left"/>
+    <xacro:steering_gazebo_v0 prefix="rear_left"/>
     <xacro:steering_gazebo_v0 prefix="rear_right"/>
-    <xacro:steering_gazebo_v0 prefix="rear_left"/>
 </robot>

Commit message: Update four_ws_robot.urdf.xacro

File: four_ws_robot_description/robots/four_ws_robot.urdf.xacro (robot description, xacro)
@@ -10,6 +10,6 @@
     <!-- Link & Joint -->
     <!-- Base -->
-    <link name="base_footprint"/> <!--link name="base_footprint"/ -->
-    <xacro:base_v0 parent="base_footprint"> <!-- xacro:base_v0 parent="base_footprint" -->
+    <link name="base_footprint"/>
+    <xacro:base_v0 parent="base_footprint">
         <origin xyz="0 0 0" rpy="0 0 0"/>
     </xacro:base_v0>

Commit message: убрал бессмысленный суффикс _v0

File: four_ws_robot_description/robots/four_ws_robot.urdf.xacro (robot description, xacro)
@@ -11,20 +11,20 @@
     <!-- Base -->
     <link name="base_footprint"/>
-    <xacro:base_v0 parent="base_footprint">
+    <xacro:base parent="base_footprint">
         <origin xyz="0 0 0" rpy="0 0 0"/>
-    </xacro:base_v0>
+    </xacro:base>
     <!-- lidar_base -->
-    <xacro:lidar_base_v0 parent="base_link">
+    <xacro:lidar_base parent="base_link">
         <origin xyz="-0.022 0 0.035" rpy="0 0 0"/>
-    </xacro:lidar_base_v0>
+    </xacro:lidar_base>
     <!-- lidar_head -->
-    <xacro:lidar_head_v0 parent="lidar_base_link">
+    <xacro:lidar_head parent="lidar_base_link">
         <origin xyz="0.022 0 0.0" rpy="0 0 0"/>
         <axis xyz="0 0 1"/>
-    </xacro:lidar_head_v0>
+    </xacro:lidar_head>
     <!-- lrf sensor -->
-    <xacro:lrf_v0 prefix = "front" parent="base_link">
+    <xacro:lrf prefix = "front" parent="base_link">
         <origin xyz="0 0 0.083" rpy="0 0 0"/>
-    </xacro:lrf_v0>
+    </xacro:lrf>
     <link name="lrf_link"/>
     <joint name="lrf_link_joint" type="fixed">
@@ -35,56 +35,56 @@
     <!-- Steering -->
     <!-- Front Right Steering -->
-    <xacro:steering_v0 prefix="front_right" parent="base_link">
+    <xacro:steering prefix="front_right" parent="base_link">
         <origin xyz="0.077 -0.031 -0.004" rpy="0 0 0"/>
         <axis xyz="0 0 1"/>
-    </xacro:steering_v0>
+    </xacro:steering>
     <!-- Front Left Steering -->
-    <xacro:steering_v0 prefix="front_left" parent="base_link">
+    <xacro:steering prefix="front_left" parent="base_link">
         <origin xyz="0.077 0.031 -0.004" rpy="0 0 0"/>
         <axis xyz="0 0 1"/>
-    </xacro:steering_v0>
+    </xacro:steering>
     <!-- Rear Right Steering -->
-    <xacro:steering_v0 prefix="rear_right" parent="base_link">
+    <xacro:steering prefix="rear_right" parent="base_link">
         <origin xyz="-0.077 -0.031 -0.004" rpy="0 0 0"/>
         <axis xyz="0 0 1"/>
-    </xacro:steering_v0>
+    </xacro:steering>
     <!-- Rear Left Steering -->
-    <xacro:steering_v0 prefix="rear_left" parent="base_link">
+    <xacro:steering prefix="rear_left" parent="base_link">
         <origin xyz="-0.077 0.031 -0.004" rpy="0 0 0"/>
         <axis xyz="0 0 1"/>
-    </xacro:steering_v0>
+    </xacro:steering>
     <!-- Wheel -->
     <!-- Front Left Wheel -->
-    <xacro:wheel_v0 prefix="fl" parent="front_left_steering_link">
+    <xacro:wheel prefix="fl" parent="front_left_steering_link">
         <origin xyz="0 0.021 -0.025" rpy="0 0 ${M_PI}"/>
         <axis xyz="0 -1 0"/>
-    </xacro:wheel_v0>
+    </xacro:wheel>
     <!-- Front Right Wheel -->
-    <xacro:wheel_v0 prefix="fr" parent="front_right_steering_link">
+    <xacro:wheel prefix="fr" parent="front_right_steering_link">
         <origin xyz="0 -0.021 -0.025" rpy="0 0 0"/>
         <axis xyz="0 1 0"/>
-    </xacro:wheel_v0>
+    </xacro:wheel>
     <!--  Rear Left Wheel -->
-    <xacro:wheel_v0 prefix="rl" parent="rear_left_steering_link">
+    <xacro:wheel prefix="rl" parent="rear_left_steering_link">
         <origin xyz="0 0.021 -0.025" rpy="0 0 ${M_PI}"/>
         <axis xyz="0 -1 0"/>
-    </xacro:wheel_v0>
+    </xacro:wheel>
     <!-- Rear Right Wheel -->
-    <xacro:wheel_v0 prefix="rr" parent="rear_right_steering_link">
+    <xacro:wheel prefix="rr" parent="rear_right_steering_link">
         <origin xyz="0 -0.021 -0.025" rpy="0 0 0"/>
         <axis xyz="0 1 0"/>
-    </xacro:wheel_v0>
+    </xacro:wheel>
     <!-- Wheel Transmission -->
-    <xacro:wheel_trans_v0 prefix="fl"/>
-    <xacro:wheel_trans_v0 prefix="fr"/>
-    <xacro:wheel_trans_v0 prefix="rl"/>
-    <xacro:wheel_trans_v0 prefix="rr"/>
+    <xacro:wheel_trans prefix="fl"/>
+    <xacro:wheel_trans prefix="fr"/>
+    <xacro:wheel_trans prefix="rl"/>
+    <xacro:wheel_trans prefix="rr"/>
     <!-- Steering Transmission -->
-    <xacro:steering_trans_v0 prefix="front_left"/>
-    <xacro:steering_trans_v0 prefix="front_right"/>
-    <xacro:steering_trans_v0 prefix="rear_left"/>
-    <xacro:steering_trans_v0 prefix="rear_right"/>
-    <!-- lider head Transmission -->
-    <xacro:lidar_trans_v0/>
+    <xacro:steering_trans prefix="front_left"/>
+    <xacro:steering_trans prefix="front_right"/>
+    <xacro:steering_trans prefix="rear_left"/>
+    <xacro:steering_trans prefix="rear_right"/>
+    <!-- lidar head Transmission -->
+    <xacro:lidar_trans/>
     <!-- Gazebo -->
     <gazebo>
@@ -102,20 +102,20 @@
     </gazebo>
     <!-- Base -->
-    <xacro:base_gazebo_v0/>
+    <xacro:base_gazebo/>
     <!-- lidar base -->
-    <xacro:lidar_base_gazebo_v0/>
+    <xacro:lidar_base_gazebo/>
     <!-- lidar head -->
-    <xacro:lidar_head_gazebo_v0/>
+    <xacro:lidar_head_gazebo/>
     <!-- lrf sensor -->
-    <xacro:lrf_gazebo_v0 prefix = "front" min_rad = "-3.14" max_rad = "3.14" min_range = "0.1" max_range = "10"/>
+    <xacro:lrf_gazebo prefix = "front" min_rad = "-3.14" max_rad = "3.14" min_range = "0.1" max_range = "10"/>
     <!-- Wheel -->
-    <xacro:wheel_gazebo_v0 prefix="fl"/>
-    <xacro:wheel_gazebo_v0 prefix="fr"/>
-    <xacro:wheel_gazebo_v0 prefix="rl"/>
-    <xacro:wheel_gazebo_v0 prefix="rr"/>
+    <xacro:wheel_gazebo prefix="fl"/>
+    <xacro:wheel_gazebo prefix="fr"/>
+    <xacro:wheel_gazebo prefix="rl"/>
+    <xacro:wheel_gazebo prefix="rr"/>
     <!-- Steering -->
-    <xacro:steering_gazebo_v0 prefix="front_left"/>
-    <xacro:steering_gazebo_v0 prefix="front_right"/>
-    <xacro:steering_gazebo_v0 prefix="rear_left"/>
-    <xacro:steering_gazebo_v0 prefix="rear_right"/>
+    <xacro:steering_gazebo prefix="front_left"/>
+    <xacro:steering_gazebo prefix="front_right"/>
+    <xacro:steering_gazebo prefix="rear_left"/>
+    <xacro:steering_gazebo prefix="rear_right"/>
 </robot>

File: four_ws_robot_description/urdf/base/base.gazebo.xacro (robot description, xacro)
@@ -1,5 +1,5 @@
 <?xml version="1.0"?>
 <robot xmlns:xacro="http://ros.org/wiki/xacro">
-    <xacro:macro name="base_gazebo_v0">
+    <xacro:macro name="base_gazebo">
         <gazebo reference="base_link">
             <selfCollide>false</selfCollide>

File: four_ws_robot_description/urdf/base/base.urdf.xacro (robot description, xacro)
@@ -2,5 +2,5 @@
 <robot xmlns:xacro="http://ros.org/wiki/xacro">
     <xacro:include filename="$(find four_ws_robot_description)/urdf/base/base.gazebo.xacro" />
-    <xacro:macro name="base_v0" params="parent *joint_origin">
+    <xacro:macro name="base" params="parent *joint_origin">
         <joint name="base_link_joint" type="fixed">
             <xacro:insert_block name="joint_origin" />

File: four_ws_robot_description/urdf/lidar_base/lidar_base.gazebo.xacro (robot description, xacro)
@@ -1,5 +1,5 @@
 <?xml version="1.0"?>
 <robot xmlns:xacro="http://ros.org/wiki/xacro">
-    <xacro:macro name="lidar_base_gazebo_v0">
+    <xacro:macro name="lidar_base_gazebo">
         <gazebo reference="lidar_base_link">
             <selfCollide>false</selfCollide>

File: four_ws_robot_description/urdf/lidar_base/lidar_base.urdf.xacro (robot description, xacro)
@@ -2,5 +2,5 @@
 <robot xmlns:xacro="http://ros.org/wiki/xacro">
     <xacro:include filename="$(find four_ws_robot_description)/urdf/lidar_base/lidar_base.gazebo.xacro" />
-    <xacro:macro name="lidar_base_v0" params="parent *joint_origin">
+    <xacro:macro name="lidar_base" params="parent *joint_origin">
         <joint name="lidar_base_link_joint" type="fixed">
             <xacro:insert_block name="joint_origin" />

File: four_ws_robot_description/urdf/lidar_head/lidar_head.gazebo.xacro (robot description, xacro)
@@ -1,5 +1,5 @@
 <?xml version="1.0"?>
 <robot xmlns:xacro="http://ros.org/wiki/xacro">
-    <xacro:macro name="lidar_head_gazebo_v0">
+    <xacro:macro name="lidar_head_gazebo">
         <gazebo reference="lidar_head_link">
             <selfCollide>false</selfCollide>

File: four_ws_robot_description/urdf/lidar_head/lidar_head.transmission.xacro (robot description, xacro)
@@ -1,5 +1,5 @@
 <?xml version="1.0"?>
 <robot xmlns:xacro="http://ros.org/wiki/xacro">
-    <xacro:macro name="lidar_trans_v0">
+    <xacro:macro name="lidar_trans">
         <transmission name="lidar_head_trans">
             <type>transmission_interface/SimpleTransmission</type>

File: four_ws_robot_description/urdf/lidar_head/lidar_head.urdf.xacro (robot description, xacro)
@@ -3,5 +3,5 @@
     <xacro:include filename="$(find four_ws_robot_description)/urdf/lidar_head/lidar_head.transmission.xacro" />
     <xacro:include filename="$(find four_ws_robot_description)/urdf/lidar_head/lidar_head.gazebo.xacro" />
-    <xacro:macro name="lidar_head_v0" params="parent *joint_origin *joint_axis">
+    <xacro:macro name="lidar_head" params="parent *joint_origin *joint_axis">
         <joint name="lidar_head_joint" type="continuous">
             <xacro:insert_block name="joint_origin" />

File: four_ws_robot_description/urdf/lrf/lrf.gazebo.xacro (robot description, xacro)
@@ -1,5 +1,5 @@
 <?xml version="1.0"?>
 <robot xmlns:xacro="http://ros.org/wiki/xacro">
-    <xacro:macro name="lrf_gazebo_v0" params="prefix min_rad max_rad min_range max_range">
+    <xacro:macro name="lrf_gazebo" params="prefix min_rad max_rad min_range max_range">
         <gazebo reference="${prefix}_lrf_link">
             <sensor type="ray" name="${prefix}_lrf_sensor">

File: four_ws_robot_description/urdf/lrf/lrf.urdf.xacro (robot description, xacro)
@@ -2,5 +2,5 @@
 <robot xmlns:xacro="http://ros.org/wiki/xacro">
     <xacro:include filename="$(find four_ws_robot_description)/urdf/lrf/lrf.gazebo.xacro" />
-    <xacro:macro name="lrf_v0" params="prefix parent *joint_origin">
+    <xacro:macro name="lrf" params="prefix parent *joint_origin">
         <joint name="${prefix}_lrf_joint" type="fixed">
             <xacro:insert_block name="joint_origin" />

File: four_ws_robot_description/urdf/suspension/suspension.gazebo.xacro (robot description, xacro)
@@ -1,9 +1,9 @@
 <?xml version="1.0"?>
 <!-- Файл "suspension.gazebo.xacro" описывает параметры модели подвески робота для симуляции
-в среде Gazebo. Он содержит макрос "steering_gazebo_v0", который определяет параметры для
+в среде Gazebo. Он содержит макрос "steering_gazebo", который определяет параметры для
 элемента "gazebo" в модели, такие как самостолкновение, коэффициенты трения между
 элементами модели и другие параметры. -->
 <robot xmlns:xacro="http://ros.org/wiki/xacro">
-    <xacro:macro name="steering_gazebo_v0" params="prefix">
+    <xacro:macro name="steering_gazebo" params="prefix">
         <gazebo reference="${prefix}_steering_link">
             <selfCollide>false</selfCollide>

File: four_ws_robot_description/urdf/suspension/suspension.transmission.xacro (robot description, xacro)
@@ -1,10 +1,10 @@
 <?xml version="1.0"?>
 <!-- Файл "suspension.transmission.xacro" определяет параметры трансмиссии робота.
-Он содержит макрос "steering_trans_v0", который определяет параметры трансмиссии,
+Он содержит макрос "steering_trans", который определяет параметры трансмиссии,
 такие как тип трансмиссии (в данном случае "transmission_interface/SimpleTransmission"),
 аппаратный интерфейс для соединения с мотором и суставом, а также
 механическое уменьшение (mechanicalReduction) для мотора. -->
 <robot xmlns:xacro="http://ros.org/wiki/xacro">
-    <xacro:macro name="steering_trans_v0" params="prefix">
+    <xacro:macro name="steering_trans" params="prefix">
         <transmission name="${prefix}_steering_trans">
             <type>transmission_interface/SimpleTransmission</type>

File: four_ws_robot_description/urdf/suspension/suspension.urdf.xacro (robot description, xacro)
@@ -1,5 +1,5 @@
 <?xml version="1.0"?>
 <!-- Файл "suspension.urdf.xacro" объединяет описания подвески робота,
-используя включения (include), и определяет макрос "steering_v0", который
+используя включения (include), и определяет макрос "steering", который
 определяет параметры соединения сустава робота. Он содержит описание соединения
 сустава, такие как тип соединения (revolute), ограничения на усилие, скорость и
@@ -8,5 +8,5 @@
     <xacro:include filename="$(find four_ws_robot_description)/urdf/suspension/suspension.transmission.xacro" />
     <xacro:include filename="$(find four_ws_robot_description)/urdf/suspension/suspension.gazebo.xacro" />
-    <xacro:macro name="steering_v0" params="prefix parent *joint_origin *joint_axis">
+    <xacro:macro name="steering" params="prefix parent *joint_origin *joint_axis">
         <joint name="${prefix}_steering_joint" type="revolute">
             <xacro:insert_block name="joint_origin" />

File: four_ws_robot_description/urdf/wheel/wheel.gazebo.xacro (robot description, xacro)
@@ -1,10 +1,10 @@
 <?xml version="1.0"?>
 <!-- Файл wheel.gazebo.xacro содержит описание модели колеса для симулятора Gazebo.
-Внутри макроса wheel_gazebo_v0 определены параметры, такие как ссылка на соответствующее
+Внутри макроса wheel_gazebo определены параметры, такие как ссылка на соответствующее
 звено колеса в URDF модели (${prefix}_wheel_link) и коэффициенты трения mu1 и mu2,
 установленные в значения 1.2. Значения коэффициентов трения mu1 и mu2 определяют трение
 между колесом и поверхностью, где робот будет симулирован в среде Gazebo. -->
 <robot xmlns:xacro="http://ros.org/wiki/xacro">
-    <xacro:macro name="wheel_gazebo_v0" params="prefix">
+    <xacro:macro name="wheel_gazebo" params="prefix">
         <gazebo reference="${prefix}_wheel_link">
             <selfCollide>false</selfCollide>

File: four_ws_robot_description/urdf/wheel/wheel.transmission.xacro (robot description, xacro)
@@ -1,5 +1,5 @@
 <?xml version="1.0"?>
 <!-- Файл wheel.transmission.xacro содержит описание трансмиссии (передачи) для колеса робота.
-Внутри макроса wheel_trans_v0 определены параметры, такие как название трансмиссии
+Внутри макроса wheel_trans определены параметры, такие как название трансмиссии
 (${prefix}_wheel_trans), тип трансмиссии (transmission_interface/SimpleTransmission),
 а также интерфейсы обмена данными с аппаратным обеспечением
@@ -7,5 +7,5 @@
 с мотором иуправления его скоростью. -->
 <robot xmlns:xacro="http://ros.org/wiki/xacro">
-    <xacro:macro name="wheel_trans_v0" params="prefix">
+    <xacro:macro name="wheel_trans" params="prefix">
         <transmission name="${prefix}_wheel_trans">
             <type>transmission_interface/SimpleTransmission</type>

File: four_ws_robot_description/urdf/wheel/wheel.urdf.xacro (robot description, xacro)
@@ -3,5 +3,5 @@
 (Unified Robot Description Format), который используется для описания геометрии,
 кинематики, инерционных свойств и других характеристик робота.
-Внутри макроса wheel_v0 определены параметры, такие как название звена колеса
+Внутри макроса wheel определены параметры, такие как название звена колеса
 (${prefix}_wheel_link), тип и ограничения соединения (<joint>),
 геометрия визуализации и столкновений колеса (<visual> и <collision>),
@@ -10,5 +10,5 @@
     <xacro:include filename="$(find four_ws_robot_description)/urdf/wheel/wheel.transmission.xacro" />
     <xacro:include filename="$(find four_ws_robot_description)/urdf/wheel/wheel.gazebo.xacro" />
-    <xacro:macro name="wheel_v0" params="prefix parent *joint_origin *joint_axis">
+    <xacro:macro name="wheel" params="prefix parent *joint_origin *joint_axis">
         <joint name="${prefix}_wheel_joint" type="continuous">
             <xacro:insert_block name="joint_origin" />
