Commit message: добавил описание камеры, добавил ее в описание робота + настроил лидар чтобы симуляция была реалистичнее

File: four_ws_robot_description/robots/four_ws_robot.urdf.xacro (robot description, xacro)
@@ -8,4 +8,5 @@
     <xacro:include filename="$(find four_ws_robot_description)/urdf/lidar_head/lidar_head.urdf.xacro"/>
     <xacro:include filename="$(find four_ws_robot_description)/urdf/lrf/lrf.urdf.xacro"/>
+    <xacro:include filename="$(find four_ws_robot_description)/urdf/camera/camera.urdf.xacro"/>
     <!-- Link & Joint -->
     <!-- Base -->
@@ -27,10 +28,8 @@
         <origin xyz="0 0 0.083" rpy="0 0 0"/>
     </xacro:lrf>
-    <link name="lrf_link"/>
-    <joint name="lrf_link_joint" type="fixed">
-        <parent link="base_link"/>
-        <child link="lrf_link"/>
-        <origin xyz="0 0 0.01" rpy="0 0 0"/>
-    </joint>
+    <!-- camera -->
+    <xacro:camera prefix="main" parent="base_link">
+        <origin xyz="0.1 0 0.0177" rpy="0 0 0"/>
+    </xacro:camera>
     <!-- Steering -->
     <!-- Front Right Steering -->
@@ -75,17 +74,37 @@
         <axis xyz="0 1 0"/>
     </xacro:wheel>
-    <!-- Wheel Transmission -->
+    <!-- base  gazebo -->
+    <xacro:base_gazebo/>
+    <!-- lidar base gazebo -->
+    <xacro:lidar_base_gazebo/>
+    <!-- lidar head gazebo -->
+    <xacro:lidar_head_gazebo/>
+    <!-- lidar head Transmission -->
+    <xacro:lidar_trans/>
+    <!-- lrf sensor -->
+    <xacro:lrf_gazebo prefix = "front" min_rad = "-${M_PI}" max_rad = "${M_PI}" min_range = "0.15" max_range = "8"/>
+    <!-- lidar head gazebo -->
+    <xacro:camera_gazebo prefix="main"/>
+    <!-- steering gazebo -->
+    <xacro:steering_gazebo prefix="front_left"/>
+    <xacro:steering_gazebo prefix="front_right"/>
+    <xacro:steering_gazebo prefix="rear_left"/>
+    <xacro:steering_gazebo prefix="rear_right"/>
+    <!-- steering transmission -->
+    <xacro:steering_trans prefix="front_left"/>
+    <xacro:steering_trans prefix="front_right"/>
+    <xacro:steering_trans prefix="rear_left"/>
+    <xacro:steering_trans prefix="rear_right"/>
+    <!-- wheel gazebo -->
+    <xacro:wheel_gazebo prefix="fl"/>
+    <xacro:wheel_gazebo prefix="fr"/>
+    <xacro:wheel_gazebo prefix="rl"/>
+    <xacro:wheel_gazebo prefix="rr"/>
+    <!-- wheel transmission gazebo -->
     <xacro:wheel_trans prefix="fl"/>
     <xacro:wheel_trans prefix="fr"/>
     <xacro:wheel_trans prefix="rl"/>
     <xacro:wheel_trans prefix="rr"/>
-    <!-- Steering Transmission -->
-    <xacro:steering_trans prefix="front_left"/>
-    <xacro:steering_trans prefix="front_right"/>
-    <xacro:steering_trans prefix="rear_left"/>
-    <xacro:steering_trans prefix="rear_right"/>
-    <!-- lidar head Transmission -->
-    <xacro:lidar_trans/>
-    <!-- Gazebo -->
+    <!-- gazebo plugins -->
     <gazebo>
         <plugin name="gazebo_ros_control" filename="libgazebo_ros_control.so"/>
@@ -101,21 +120,3 @@
         </plugin>
     </gazebo>
-    <!-- Base -->
-    <xacro:base_gazebo/>
-    <!-- lidar base -->
-    <xacro:lidar_base_gazebo/>
-    <!-- lidar head -->
-    <xacro:lidar_head_gazebo/>
-    <!-- lrf sensor -->
-    <xacro:lrf_gazebo prefix = "front" min_rad = "-3.14" max_rad = "3.14" min_range = "0.1" max_range = "10"/>
-    <!-- Wheel -->
-    <xacro:wheel_gazebo prefix="fl"/>
-    <xacro:wheel_gazebo prefix="fr"/>
-    <xacro:wheel_gazebo prefix="rl"/>
-    <xacro:wheel_gazebo prefix="rr"/>
-    <!-- Steering -->
-    <xacro:steering_gazebo prefix="front_left"/>
-    <xacro:steering_gazebo prefix="front_right"/>
-    <xacro:steering_gazebo prefix="rear_left"/>
-    <xacro:steering_gazebo prefix="rear_right"/>
 </robot>

File: four_ws_robot_description/urdf/lrf/lrf.gazebo.xacro (robot description, xacro)
@@ -6,5 +6,5 @@
                 <pose>0 0 0 0 0 0</pose>
                 <visualize>true</visualize>
-                <update_rate>40</update_rate>
+                <update_rate>10</update_rate>
                 <ray>
                     <scan>

Commit message: еще доработал файлы описания робота и добавил требуемый пакет

File: four_ws_robot_description/robots/four_ws_robot.urdf.xacro (robot description, xacro)
@@ -1,112 +1,111 @@
 <?xml version="1.0"?>
-<robot name="four_ws_robot" xmlns:xacro="http://ros.org/wiki/xacro">
-    <xacro:property name="M_PI" value="3.14159274"/>
-    <xacro:include filename="$(find four_ws_robot_description)/urdf/base/base.urdf.xacro"/>
-    <xacro:include filename="$(find four_ws_robot_description)/urdf/suspension/suspension.urdf.xacro"/>
-    <xacro:include filename="$(find four_ws_robot_description)/urdf/wheel/wheel.urdf.xacro"/>
-    <xacro:include filename="$(find four_ws_robot_description)/urdf/lidar_base/lidar_base.urdf.xacro"/>
-    <xacro:include filename="$(find four_ws_robot_description)/urdf/lidar_head/lidar_head.urdf.xacro"/>
-    <xacro:include filename="$(find four_ws_robot_description)/urdf/lrf/lrf.urdf.xacro"/>
-    <xacro:include filename="$(find four_ws_robot_description)/urdf/camera/camera.urdf.xacro"/>
-    <!-- Link & Joint -->
+<robot xmlns:xacro="http://ros.org/wiki/xacro" name="four_ws_robot">
+    <xacro:property name="M_PI" value="3.14159274" />
+    <xacro:include filename="$(find four_ws_robot_description)/urdf/base/base.urdf.xacro" />
+    <xacro:include filename="$(find four_ws_robot_description)/urdf/base/base.gazebo.xacro" />
+    <xacro:include filename="$(find four_ws_robot_description)/urdf/camera/camera.urdf.xacro" />
+    <xacro:include filename="$(find four_ws_robot_description)/urdf/camera/camera.gazebo.xacro" />
+    <xacro:include filename="$(find four_ws_robot_description)/urdf/lidar_base/lidar_base.urdf.xacro" />
+    <xacro:include filename="$(find four_ws_robot_description)/urdf/lidar_base/lidar_base.gazebo.xacro" />
+    <xacro:include filename="$(find four_ws_robot_description)/urdf/lidar_head/lidar_head.urdf.xacro" />
+    <xacro:include filename="$(find four_ws_robot_description)/urdf/lidar_head/lidar_head.gazebo.xacro" />
+    <xacro:include filename="$(find four_ws_robot_description)/urdf/lidar_head/lidar_head.transmission.xacro" />
+    <xacro:include filename="$(find four_ws_robot_description)/urdf/lrf/lrf.urdf.xacro" />
+    <xacro:include filename="$(find four_ws_robot_description)/urdf/lrf/lrf.gazebo.xacro" />
+    <xacro:include filename="$(find four_ws_robot_description)/urdf/suspension/suspension.urdf.xacro" />
+    <xacro:include filename="$(find four_ws_robot_description)/urdf/suspension/suspension.gazebo.xacro" />
+    <xacro:include filename="$(find four_ws_robot_description)/urdf/suspension/suspension.transmission.xacro" />
+    <xacro:include filename="$(find four_ws_robot_description)/urdf/wheel/wheel.urdf.xacro" />
+    <xacro:include filename="$(find four_ws_robot_description)/urdf/wheel/wheel.gazebo.xacro" />
+    <xacro:include filename="$(find four_ws_robot_description)/urdf/wheel/wheel.transmission.xacro" />
     <!-- Base -->
-    <link name="base_footprint"/>
+    <link name="base_footprint" />
     <xacro:base parent="base_footprint">
-        <origin xyz="0 0 0" rpy="0 0 0"/>
+        <origin xyz="0 0 0" rpy="0 0 0" />
     </xacro:base>
+    <xacro:base_gazebo />
     <!-- lidar_base -->
     <xacro:lidar_base parent="base_link">
-        <origin xyz="-0.022 0 0.035" rpy="0 0 0"/>
+        <origin xyz="-0.022 0 0.035" rpy="0 0 0" />
     </xacro:lidar_base>
+    <xacro:lidar_base_gazebo />
     <!-- lidar_head -->
     <xacro:lidar_head parent="lidar_base_link">
-        <origin xyz="0.022 0 0.0" rpy="0 0 0"/>
-        <axis xyz="0 0 1"/>
+        <origin xyz="0.022 0 0.0" rpy="0 0 0" />
+        <axis xyz="0 0 1" />
     </xacro:lidar_head>
+    <xacro:lidar_head_gazebo />
+    <xacro:lidar_head_trans />
     <!-- lrf sensor -->
-    <xacro:lrf prefix = "front" parent="base_link">
-        <origin xyz="0 0 0.083" rpy="0 0 0"/>
+    <xacro:lrf prefix="front" parent="base_link">
+        <origin xyz="0 0 0.083" rpy="0 0 0" />
     </xacro:lrf>
+    <xacro:lrf_gazebo prefix="front" min_rad="-${M_PI}" max_rad="${M_PI}" min_range="0.15" max_range="8" />
     <!-- camera -->
-    <xacro:camera prefix="main" parent="base_link">
-        <origin xyz="0.1 0 0.0177" rpy="0 0 0"/>
+    <xacro:camera prefix="front" parent="base_link">
+        <origin xyz="0.1 0 0.0177" rpy="0 0 0" />
     </xacro:camera>
+    <xacro:camera_gazebo prefix="front" />
     <!-- Steering -->
     <!-- Front Right Steering -->
     <xacro:steering prefix="front_right" parent="base_link">
-        <origin xyz="0.077 -0.031 -0.004" rpy="0 0 0"/>
-        <axis xyz="0 0 1"/>
+        <origin xyz="0.077 -0.031 -0.004" rpy="0 0 0" />
+        <axis xyz="0 0 1" />
     </xacro:steering>
+    <xacro:steering_gazebo prefix="front_right" />
+    <xacro:steering_trans prefix="front_right" />
     <!-- Front Left Steering -->
     <xacro:steering prefix="front_left" parent="base_link">
-        <origin xyz="0.077 0.031 -0.004" rpy="0 0 0"/>
-        <axis xyz="0 0 1"/>
+        <origin xyz="0.077 0.031 -0.004" rpy="0 0 0" />
+        <axis xyz="0 0 1" />
     </xacro:steering>
+    <xacro:steering_gazebo prefix="front_left" />
+    <xacro:steering_trans prefix="front_left" />
     <!-- Rear Right Steering -->
     <xacro:steering prefix="rear_right" parent="base_link">
-        <origin xyz="-0.077 -0.031 -0.004" rpy="0 0 0"/>
-        <axis xyz="0 0 1"/>
+        <origin xyz="-0.077 -0.031 -0.004" rpy="0 0 0" />
+        <axis xyz="0 0 1" />
     </xacro:steering>
+    <xacro:steering_gazebo prefix="rear_right" />
+    <xacro:steering_trans prefix="rear_right" />
     <!-- Rear Left Steering -->
     <xacro:steering prefix="rear_left" parent="base_link">
-        <origin xyz="-0.077 0.031 -0.004" rpy="0 0 0"/>
-        <axis xyz="0 0 1"/>
+        <origin xyz="-0.077 0.031 -0.004" rpy="0 0 0" />
+        <axis xyz="0 0 1" />
     </xacro:steering>
+    <xacro:steering_gazebo prefix="rear_left" />
+    <xacro:steering_trans prefix="rear_left" />
     <!-- Wheel -->
     <!-- Front Left Wheel -->
     <xacro:wheel prefix="fl" parent="front_left_steering_link">
-        <origin xyz="0 0.021 -0.025" rpy="0 0 ${M_PI}"/>
-        <axis xyz="0 -1 0"/>
+        <origin xyz="0 0.021 -0.025" rpy="0 0 ${M_PI}" />
+        <axis xyz="0 -1 0" />
     </xacro:wheel>
+    <xacro:wheel_gazebo prefix="fl" />
+    <xacro:wheel_trans prefix="fl" />
     <!-- Front Right Wheel -->
     <xacro:wheel prefix="fr" parent="front_right_steering_link">
-        <origin xyz="0 -0.021 -0.025" rpy="0 0 0"/>
-        <axis xyz="0 1 0"/>
+        <origin xyz="0 -0.021 -0.025" rpy="0 0 0" />
+        <axis xyz="0 1 0" />
     </xacro:wheel>
+    <xacro:wheel_gazebo prefix="fr" />
+    <xacro:wheel_trans prefix="fr" />
     <!--  Rear Left Wheel -->
     <xacro:wheel prefix="rl" parent="rear_left_steering_link">
-        <origin xyz="0 0.021 -0.025" rpy="0 0 ${M_PI}"/>
-        <axis xyz="0 -1 0"/>
+        <origin xyz="0 0.021 -0.025" rpy="0 0 ${M_PI}" />
+        <axis xyz="0 -1 0" />
     </xacro:wheel>
+    <xacro:wheel_gazebo prefix="rl" />
+    <xacro:wheel_trans prefix="rl" />
     <!-- Rear Right Wheel -->
     <xacro:wheel prefix="rr" parent="rear_right_steering_link">
-        <origin xyz="0 -0.021 -0.025" rpy="0 0 0"/>
-        <axis xyz="0 1 0"/>
+        <origin xyz="0 -0.021 -0.025" rpy="0 0 0" />
+        <axis xyz="0 1 0" />
     </xacro:wheel>
-    <!-- base  gazebo -->
-    <xacro:base_gazebo/>
-    <!-- lidar base gazebo -->
-    <xacro:lidar_base_gazebo/>
-    <!-- lidar head gazebo -->
-    <xacro:lidar_head_gazebo/>
-    <!-- lidar head Transmission -->
-    <xacro:lidar_trans/>
-    <!-- lrf sensor -->
-    <xacro:lrf_gazebo prefix = "front" min_rad = "-${M_PI}" max_rad = "${M_PI}" min_range = "0.15" max_range = "8"/>
-    <!-- lidar head gazebo -->
-    <xacro:camera_gazebo prefix="main"/>
-    <!-- steering gazebo -->
-    <xacro:steering_gazebo prefix="front_left"/>
-    <xacro:steering_gazebo prefix="front_right"/>
-    <xacro:steering_gazebo prefix="rear_left"/>
-    <xacro:steering_gazebo prefix="rear_right"/>
-    <!-- steering transmission -->
-    <xacro:steering_trans prefix="front_left"/>
-    <xacro:steering_trans prefix="front_right"/>
-    <xacro:steering_trans prefix="rear_left"/>
-    <xacro:steering_trans prefix="rear_right"/>
-    <!-- wheel gazebo -->
-    <xacro:wheel_gazebo prefix="fl"/>
-    <xacro:wheel_gazebo prefix="fr"/>
-    <xacro:wheel_gazebo prefix="rl"/>
-    <xacro:wheel_gazebo prefix="rr"/>
-    <!-- wheel transmission gazebo -->
-    <xacro:wheel_trans prefix="fl"/>
-    <xacro:wheel_trans prefix="fr"/>
-    <xacro:wheel_trans prefix="rl"/>
-    <xacro:wheel_trans prefix="rr"/>
+    <xacro:wheel_gazebo prefix="rr" />
+    <xacro:wheel_trans prefix="rr" />
     <!-- gazebo plugins -->
     <gazebo>
-        <plugin name="gazebo_ros_control" filename="libgazebo_ros_control.so"/>
+        <plugin name="gazebo_ros_control" filename="libgazebo_ros_control.so" />
         <plugin name="p3d_base_controller" filename="libgazebo_ros_p3d.so">
             <alwaysOn>true</alwaysOn>

File: four_ws_robot_description/urdf/camera/camera.gazebo.xacro (robot description, xacro)
@@ -1,3 +1,3 @@
-<?xml version="1.0" encoding="UTF-8"?>
+<?xml version="1.0"?>
 <robot xmlns:xacro="http://ros.org/wiki/xacro">
     <xacro:macro name="camera_gazebo" params="prefix">
@@ -8,5 +8,5 @@
                 <update_rate>10</update_rate>
                 <camera>
-                    <horizontal_fov>1.089</horizontal_fov>
+                    <horizontal_fov>1.3962634</horizontal_fov>
                     <image>
                         <format>R8G8B8</format>
@@ -18,7 +18,22 @@
                         <far>100</far>
                     </clip>
+                    <noise>
+                        <type>gaussian</type>
+                        <mean>0.0</mean>
+                        <stddev>0.01</stddev>
+                    </noise>
                 </camera>
                 <plugin name="camera_controller" filename="libgazebo_ros_camera.so">
+                    <updateRate>0.0</updateRate>
+                    <cameraName>camera</cameraName>
+                    <imageTopicName>image_raw</imageTopicName>
+                    <cameraInfoTopicName>camera_info</cameraInfoTopicName>
                     <frameName>${prefix}_camera_link</frameName>
+                    <hackBaseline>0.07</hackBaseline>
+                    <distortionK1>0.0</distortionK1>
+                    <distortionK2>0.0</distortionK2>
+                    <distortionK3>0.0</distortionK3>
+                    <distortionT1>0.0</distortionT1>
+                    <distortionT2>0.0</distortionT2>
                 </plugin>
             </sensor>

File: four_ws_robot_description/urdf/camera/camera.urdf.xacro (robot description, xacro)
@@ -1,5 +1,4 @@
-<?xml version="1.0" encoding="UTF-8"?>
-<robot xmlns:xacro="http://ros.org/wiki/xacro" name="delirobo">
-    <xacro:include filename="$(find four_ws_robot_description)/urdf/camera/camera.gazebo.xacro" />
+<?xml version="1.0"?>
+<robot xmlns:xacro="http://ros.org/wiki/xacro">
     <xacro:macro name="camera" params="prefix parent *joint_origin">
         <joint name="${prefix}_camera_joint" type="fixed">

File: four_ws_robot_description/urdf/lidar_base/lidar_base.urdf.xacro (robot description, xacro)
@@ -1,7 +1,6 @@
 <?xml version="1.0"?>
 <robot xmlns:xacro="http://ros.org/wiki/xacro">
-    <xacro:include filename="$(find four_ws_robot_description)/urdf/lidar_base/lidar_base.gazebo.xacro" />
     <xacro:macro name="lidar_base" params="parent *joint_origin">
-        <joint name="lidar_base_link_joint" type="fixed">
+        <joint name="lidar_base_joint" type="fixed">
             <xacro:insert_block name="joint_origin" />
             <parent link="${parent}" />

File: four_ws_robot_description/urdf/lidar_head/lidar_head.transmission.xacro (robot description, xacro)
@@ -1,5 +1,5 @@
 <?xml version="1.0"?>
 <robot xmlns:xacro="http://ros.org/wiki/xacro">
-    <xacro:macro name="lidar_trans">
+    <xacro:macro name="lidar_head_trans">
         <transmission name="lidar_head_trans">
             <type>transmission_interface/SimpleTransmission</type>

File: four_ws_robot_description/urdf/lidar_head/lidar_head.urdf.xacro (robot description, xacro)
@@ -1,6 +1,4 @@
 <?xml version="1.0"?>
 <robot xmlns:xacro="http://ros.org/wiki/xacro">
-    <xacro:include filename="$(find four_ws_robot_description)/urdf/lidar_head/lidar_head.transmission.xacro" />
-    <xacro:include filename="$(find four_ws_robot_description)/urdf/lidar_head/lidar_head.gazebo.xacro" />
     <xacro:macro name="lidar_head" params="parent *joint_origin *joint_axis">
         <joint name="lidar_head_joint" type="continuous">

File: four_ws_robot_description/urdf/lrf/lrf.urdf.xacro (robot description, xacro)
@@ -1,5 +1,4 @@
 <?xml version="1.0"?>
 <robot xmlns:xacro="http://ros.org/wiki/xacro">
-    <xacro:include filename="$(find four_ws_robot_description)/urdf/lrf/lrf.gazebo.xacro" />
     <xacro:macro name="lrf" params="prefix parent *joint_origin">
         <joint name="${prefix}_lrf_joint" type="fixed">

File: four_ws_robot_description/urdf/suspension/suspension.urdf.xacro (robot description, xacro)
@@ -1,6 +1,4 @@
 <?xml version="1.0"?>
 <robot xmlns:xacro="http://ros.org/wiki/xacro">
-    <xacro:include filename="$(find four_ws_robot_description)/urdf/suspension/suspension.transmission.xacro" />
-    <xacro:include filename="$(find four_ws_robot_description)/urdf/suspension/suspension.gazebo.xacro" />
     <xacro:macro name="steering" params="prefix parent *joint_origin *joint_axis">
         <joint name="${prefix}_steering_joint" type="revolute">

File: four_ws_robot_description/urdf/wheel/wheel.urdf.xacro (robot description, xacro)
@@ -1,6 +1,4 @@
 <?xml version="1.0"?>
 <robot xmlns:xacro="http://ros.org/wiki/xacro">
-    <xacro:include filename="$(find four_ws_robot_description)/urdf/wheel/wheel.transmission.xacro" />
-    <xacro:include filename="$(find four_ws_robot_description)/urdf/wheel/wheel.gazebo.xacro" />
     <xacro:macro name="wheel" params="prefix parent *joint_origin *joint_axis">
         <joint name="${prefix}_wheel_joint" type="continuous">

Commit message: убрал логику врещений lidar_head

File: four_ws_robot_description/robots/four_ws_robot.urdf.xacro (robot description, xacro)
@@ -10,5 +10,4 @@
     <xacro:include filename="$(find four_ws_robot_description)/urdf/lidar_head/lidar_head.urdf.xacro" />
     <xacro:include filename="$(find four_ws_robot_description)/urdf/lidar_head/lidar_head.gazebo.xacro" />
-    <xacro:include filename="$(find four_ws_robot_description)/urdf/lidar_head/lidar_head.transmission.xacro" />
     <xacro:include filename="$(find four_ws_robot_description)/urdf/lrf/lrf.urdf.xacro" />
     <xacro:include filename="$(find four_ws_robot_description)/urdf/lrf/lrf.gazebo.xacro" />
@@ -33,8 +32,6 @@
     <xacro:lidar_head parent="lidar_base_link">
         <origin xyz="0.022 0 0.0" rpy="0 0 0" />
-        <axis xyz="0 0 1" />
     </xacro:lidar_head>
     <xacro:lidar_head_gazebo />
-    <xacro:lidar_head_trans />
     <!-- lrf sensor -->
     <xacro:lrf prefix="front" parent="base_link">

File: four_ws_robot_description/urdf/lidar_head/lidar_head.urdf.xacro (robot description, xacro)
@@ -1,11 +1,9 @@
 <?xml version="1.0"?>
 <robot xmlns:xacro="http://ros.org/wiki/xacro">
-    <xacro:macro name="lidar_head" params="parent *joint_origin *joint_axis">
-        <joint name="lidar_head_joint" type="continuous">
+    <xacro:macro name="lidar_head" params="parent *joint_origin">
+        <joint name="lidar_head_joint" type="fixed">
             <xacro:insert_block name="joint_origin" />
             <parent link="${parent}" />
             <child link="lidar_head_link" />
-            <limit effort="1.5" velocity="20" />
-            <xacro:insert_block name="joint_axis" />
         </joint>
         <link name="lidar_head_link">
