Commit message: link, который формирует лазерный скан, теперь называется lidar_scan и топик теперь называется /scan

File: four_ws_robot_description/robots/four_ws_robot.urdf.xacro (robot description, xacro)
@@ -10,6 +10,6 @@
     <xacro:include filename="$(find four_ws_robot_description)/urdf/lidar_head/lidar_head.urdf.xacro" />
     <xacro:include filename="$(find four_ws_robot_description)/urdf/lidar_head/lidar_head.gazebo.xacro" />
-    <xacro:include filename="$(find four_ws_robot_description)/urdf/lrf/lrf.urdf.xacro" />
-    <xacro:include filename="$(find four_ws_robot_description)/urdf/lrf/lrf.gazebo.xacro" />
+    <xacro:include filename="$(find four_ws_robot_description)/urdf/lidar_scan/lidar_scan.urdf.xacro" />
+    <xacro:include filename="$(find four_ws_robot_description)/urdf/lidar_scan/lidar_scan.gazebo.xacro" />
     <xacro:include filename="$(find four_ws_robot_description)/urdf/suspension/suspension.urdf.xacro" />
     <xacro:include filename="$(find four_ws_robot_description)/urdf/suspension/suspension.gazebo.xacro" />
@@ -34,9 +34,9 @@
     </xacro:lidar_head>
     <xacro:lidar_head_gazebo />
-    <!-- lrf sensor -->
-    <xacro:lrf prefix="front" parent="base_link">
+    <!-- lidar_scan sensor -->
+    <xacro:lidar_scan parent="base_link">
         <origin xyz="0 0 0.083" rpy="0 0 0" />
-    </xacro:lrf>
-    <xacro:lrf_gazebo prefix="front" min_rad="-${M_PI}" max_rad="${M_PI}" min_range="0.15" max_range="8" />
+    </xacro:lidar_scan>
+    <xacro:lidar_scan_gazebo min_rad="-${M_PI}" max_rad="${M_PI}" min_range="0.15" max_range="8" />
     <!-- camera -->
     <xacro:camera prefix="front" parent="base_link">
@@ -107,5 +107,5 @@
         <plugin name="p3d_base_controller" filename="libgazebo_ros_p3d.so">
             <alwaysOn>true</alwaysOn>
-            <updateRate>10.0</updateRate>
+            <updateRate>10</updateRate>
             <bodyName>base_link</bodyName>
             <topicName>ground_truth/state</topicName>

File: four_ws_robot_description/urdf/lidar_scan/lidar_scan.gazebo.xacro (robot description, xacro)
@@ -1,10 +1,10 @@
 <?xml version="1.0"?>
 <robot xmlns:xacro="http://ros.org/wiki/xacro">
-    <xacro:macro name="lrf_gazebo" params="prefix min_rad max_rad min_range max_range">
-        <gazebo reference="${prefix}_lrf_link">
-            <sensor type="ray" name="${prefix}_lrf_sensor">
+    <xacro:macro name="lidar_scan_gazebo" params="min_rad max_rad min_range max_range">
+        <gazebo reference="lidar_scan_link">
+            <sensor type="ray" name="lidar_scan_sensor">
                 <pose>0 0 0 0 0 0</pose>
                 <visualize>true</visualize>
-                <update_rate>10</update_rate>
+                <update_rate>5</update_rate>
                 <ray>
                     <scan>
@@ -27,8 +27,7 @@
                     </noise>
                 </ray>
-                <plugin name="gazebo_ros_${prefix}_lrf_controller" filename="libgazebo_ros_laser.so">
-                    <topicName>${prefix}/scan</topicName>
-                    <!-- do ont set it to base_scan -->
-                    <frameName>${prefix}_lrf_link</frameName>
+                <plugin name="gazebo_ros_lidar_scan_controller" filename="libgazebo_ros_laser.so">
+                    <topicName>scan</topicName>
+                    <frameName>lidar_scan_link</frameName>
                 </plugin>
             </sensor>

Commit message: поднял немного сенсор

File: four_ws_robot_description/robots/four_ws_robot.urdf.xacro (robot description, xacro)
@@ -34,7 +34,7 @@
     </xacro:lidar_head>
     <xacro:lidar_head_gazebo />
-    <!-- lidar_scan sensor -->
+    <!-- lidar_scan -->
     <xacro:lidar_scan parent="base_link">
-        <origin xyz="0 0 0.083" rpy="0 0 0" />
+        <origin xyz="0 0 0.084" rpy="0 0 0" />
     </xacro:lidar_scan>
     <xacro:lidar_scan_gazebo min_rad="-${M_PI}" max_rad="${M_PI}" min_range="0.15" max_range="8" />

Commit message: убрал link "lidar_scan", теперь плагин лидара стоит в  "lidar_head"; осталась проблема со смешением основной точки скана

File: four_ws_robot_description/robots/four_ws_robot.urdf.xacro (robot description, xacro)
@@ -10,6 +10,4 @@
     <xacro:include filename="$(find four_ws_robot_description)/urdf/lidar_head/lidar_head.urdf.xacro" />
     <xacro:include filename="$(find four_ws_robot_description)/urdf/lidar_head/lidar_head.gazebo.xacro" />
-    <xacro:include filename="$(find four_ws_robot_description)/urdf/lidar_scan/lidar_scan.urdf.xacro" />
-    <xacro:include filename="$(find four_ws_robot_description)/urdf/lidar_scan/lidar_scan.gazebo.xacro" />
     <xacro:include filename="$(find four_ws_robot_description)/urdf/suspension/suspension.urdf.xacro" />
     <xacro:include filename="$(find four_ws_robot_description)/urdf/suspension/suspension.gazebo.xacro" />
@@ -33,10 +31,5 @@
         <origin xyz="0.022 0 0.0" rpy="0 0 0" />
     </xacro:lidar_head>
-    <xacro:lidar_head_gazebo />
-    <!-- lidar_scan -->
-    <xacro:lidar_scan parent="base_link">
-        <origin xyz="0 0 0.084" rpy="0 0 0" />
-    </xacro:lidar_scan>
-    <xacro:lidar_scan_gazebo min_rad="-${M_PI}" max_rad="${M_PI}" min_range="0.15" max_range="8" />
+    <xacro:lidar_head_gazebo min_rad="-${M_PI}" max_rad="${M_PI}" min_range="0.15" max_range="8" />
     <!-- camera -->
     <xacro:camera prefix="front" parent="base_link">

File: four_ws_robot_description/urdf/lidar_head/lidar_head.gazebo.xacro (robot description, xacro)
@@ -1,9 +1,38 @@
 <?xml version="1.0"?>
 <robot xmlns:xacro="http://ros.org/wiki/xacro">
-    <xacro:macro name="lidar_head_gazebo">
+    <xacro:macro name="lidar_head_gazebo" params="min_rad max_rad min_range max_range">
         <gazebo reference="lidar_head_link">
             <selfCollide>false</selfCollide>
             <mu1 value="0.05" />
             <mu2 value="0.05" />
+            <sensor type="ray" name="lidar_head_sensor">
+                <pose>0 0 0.049 0 0 0</pose>
+                <visualize>true</visualize>
+                <update_rate>5</update_rate>
+                <ray>
+                    <scan>
+                        <horizontal>
+                            <samples>720</samples>
+                            <resolution>1</resolution>
+                            <min_angle>${min_rad}</min_angle>
+                            <max_angle>${max_rad}</max_angle>
+                        </horizontal>
+                    </scan>
+                    <range>
+                        <min>${min_range}</min>
+                        <max>${max_range}</max>
+                        <resolution>0.01</resolution>
+                    </range>
+                    <noise>
+                        <type>gaussian</type>
+                        <mean>0.0</mean>
+                        <stddev>0.03</stddev>
+                    </noise>
+                </ray>
+                <plugin name="gazebo_ros_lidar_head_controller" filename="libgazebo_ros_laser.so">
+                    <topicName>scan</topicName>
+                    <frameName>lidar_head_link</frameName>
+                </plugin>
+            </sensor>
         </gazebo>
     </xacro:macro>

Commit message: теперь base_footprint точно под base_link, а не сопадает с ним

File: four_ws_robot_description/robots/four_ws_robot.urdf.xacro (robot description, xacro)
@@ -16,8 +16,10 @@
     <xacro:include filename="$(find four_ws_robot_description)/urdf/wheel/wheel.gazebo.xacro" />
     <xacro:include filename="$(find four_ws_robot_description)/urdf/wheel/wheel.transmission.xacro" />
+    <!-- base_footprint -->
+    <link name="base_footprint" />
+    <gazebo reference="base_footprint" />
     <!-- base -->
-    <link name="base_footprint" />
     <xacro:base parent="base_footprint">
-        <origin xyz="0 0 0" rpy="0 0 0" />
+        <origin xyz="0 0 0.055" rpy="0 0 0" />
     </xacro:base>
     <xacro:base_gazebo />
@@ -33,8 +35,8 @@
     <xacro:lidar_head_gazebo min_rad="-${M_PI}" max_rad="${M_PI}" min_range="0.15" max_range="8" />
     <!-- camera -->
-    <xacro:camera prefix="front" parent="base_link">
+    <xacro:camera parent="base_link">
         <origin xyz="0.1 0 0.0177" rpy="0 0 0" />
     </xacro:camera>
-    <xacro:camera_gazebo prefix="front" />
+    <xacro:camera_gazebo />
     <!-- steering -->
     <!-- front right -->

File: four_ws_robot_description/urdf/camera/camera.gazebo.xacro (robot description, xacro)
@@ -1,7 +1,7 @@
 <?xml version="1.0"?>
 <robot xmlns:xacro="http://ros.org/wiki/xacro">
-    <xacro:macro name="camera_gazebo" params="prefix">
-        <gazebo reference="${prefix}_camera_link">
-            <sensor type="camera" name="${prefix}">
+    <xacro:macro name="camera_gazebo">
+        <gazebo reference="camera_link">
+            <sensor type="camera" name="camera">
                 <pose>0 0 0 0 0 0</pose>
                 <visualize>true</visualize>
@@ -29,5 +29,5 @@
                     <imageTopicName>image_raw</imageTopicName>
                     <cameraInfoTopicName>camera_info</cameraInfoTopicName>
-                    <frameName>${prefix}_camera_link</frameName>
+                    <frameName>camera_link</frameName>
                     <hackBaseline>0.07</hackBaseline>
                     <distortionK1>0.0</distortionK1>

File: four_ws_robot_description/urdf/camera/camera.urdf.xacro (robot description, xacro)
@@ -1,11 +1,11 @@
 <?xml version="1.0"?>
 <robot xmlns:xacro="http://ros.org/wiki/xacro">
-    <xacro:macro name="camera" params="prefix parent *joint_origin">
-        <joint name="${prefix}_camera_joint" type="fixed">
+    <xacro:macro name="camera" params="parent *joint_origin">
+        <joint name="camera_joint" type="fixed">
             <xacro:insert_block name="joint_origin" />
             <parent link="${parent}" />
-            <child link="${prefix}_camera_link" />
+            <child link="camera_link" />
         </joint>
-        <link name="${prefix}_camera_link">
+        <link name="camera_link">
             <visual>
                 <geometry>

Commit message: подредачил файлы описания робота, переименовал файлы подвески и убрал постфикс "_link" в описании моделек

File: four_ws_robot_description/robots/four_ws_robot.urdf.xacro (robot description, xacro)
@@ -10,7 +10,7 @@
     <xacro:include filename="$(find four_ws_robot_description)/urdf/lidar_head/lidar_head.urdf.xacro" />
     <xacro:include filename="$(find four_ws_robot_description)/urdf/lidar_head/lidar_head.gazebo.xacro" />
-    <xacro:include filename="$(find four_ws_robot_description)/urdf/suspension/suspension.urdf.xacro" />
-    <xacro:include filename="$(find four_ws_robot_description)/urdf/suspension/suspension.gazebo.xacro" />
-    <xacro:include filename="$(find four_ws_robot_description)/urdf/suspension/suspension.transmission.xacro" />
+    <xacro:include filename="$(find four_ws_robot_description)/urdf/steering/steering.urdf.xacro" />
+    <xacro:include filename="$(find four_ws_robot_description)/urdf/steering/steering.gazebo.xacro" />
+    <xacro:include filename="$(find four_ws_robot_description)/urdf/steering/steering.transmission.xacro" />
     <xacro:include filename="$(find four_ws_robot_description)/urdf/wheel/wheel.urdf.xacro" />
     <xacro:include filename="$(find four_ws_robot_description)/urdf/wheel/wheel.gazebo.xacro" />

File: four_ws_robot_description/urdf/base/base.urdf.xacro (robot description, xacro)
@@ -11,5 +11,5 @@
             <visual>
                 <geometry>
-                    <mesh filename="package://four_ws_robot_description/meshes/DAE/base/base_link.dae" />
+                    <mesh filename="package://four_ws_robot_description/meshes/DAE/base/base.dae" />
                 </geometry>
                 <origin xyz="0.0 0.0 0.0" />
@@ -17,5 +17,5 @@
             <collision>
                 <geometry>
-                    <mesh filename="package://four_ws_robot_description/meshes/STL/base/base_link.stl" />
+                    <mesh filename="package://four_ws_robot_description/meshes/STL/base/base.stl" />
                 </geometry>
                 <origin xyz="0.0 0.0 0.0" />

File: four_ws_robot_description/urdf/camera/camera.urdf.xacro (robot description, xacro)
@@ -10,5 +10,5 @@
             <visual>
                 <geometry>
-                    <mesh filename="package://four_ws_robot_description/meshes/DAE/sensors/camera/camera.dae" />
+                    <mesh filename="package://four_ws_robot_description/meshes/DAE/camera/camera.dae" />
                 </geometry>
                 <origin xyz="0.0 0.0 0.0" />
@@ -16,5 +16,5 @@
             <collision>
                 <geometry>
-                    <mesh filename="package://four_ws_robot_description/meshes/STL/sensors/camera/camera.stl" />
+                    <mesh filename="package://four_ws_robot_description/meshes/STL/camera/camera.stl" />
                 </geometry>
                 <origin xyz="0.0 0.0 0.0" />

File: four_ws_robot_description/urdf/steering/steering.urdf.xacro (robot description, xacro)
@@ -12,5 +12,5 @@
             <visual>
                 <geometry>
-                    <mesh filename="package://four_ws_robot_description/meshes/DAE/suspension/${prefix}_link.dae" />
+                    <mesh filename="package://four_ws_robot_description/meshes/DAE/steering/${prefix}_steering.dae" />
                 </geometry>
                 <origin xyz="0.0 0.0 0.0" />
@@ -18,5 +18,5 @@
             <collision>
                 <geometry>
-                    <mesh filename="package://four_ws_robot_description/meshes/STL/suspension/sus_link.stl" />
+                    <mesh filename="package://four_ws_robot_description/meshes/STL/steering/steering.stl" />
                 </geometry>
                 <origin xyz="0.0 0.0 0.0" />

File: four_ws_robot_description/urdf/wheel/wheel.urdf.xacro (robot description, xacro)
@@ -12,5 +12,5 @@
             <visual>
                 <geometry>
-                    <mesh filename="package://four_ws_robot_description/meshes/DAE/wheel/wheel_link.dae" />
+                    <mesh filename="package://four_ws_robot_description/meshes/DAE/wheel/wheel.dae" />
                 </geometry>
                 <origin xyz="0.0 0.0 0.0" />
@@ -18,5 +18,5 @@
             <collision>
                 <geometry>
-                    <mesh filename="package://four_ws_robot_description/meshes/STL/wheel/robot_wheel.stl" />
+                    <mesh filename="package://four_ws_robot_description/meshes/STL/wheel/wheel.stl" />
                 </geometry>
                 <origin xyz="0.0 0.0 0.0" />

Commit message: исправил центры масс у деталей, убрал joint_state_publisher т к данные о положении сочленений будем брать из симулятора

File: four_ws_robot_description/robots/four_ws_robot.urdf.xacro (robot description, xacro)
@@ -100,5 +100,6 @@
     <gazebo>
         <!-- gazebo plugins -->
-        <plugin name="gazebo_ros_control" filename="libgazebo_ros_control.so" />
+        <plugin name="gazebo_ros_control" filename="libgazebo_ros_control.so">
+        </plugin>
         <!-- plugin that publishes the position of the coordinate system "bodyName"
         relative to "frameName" in the topic "ground_truth/state" -->

File: four_ws_robot_description/urdf/base/base.urdf.xacro (robot description, xacro)
@@ -12,5 +12,5 @@
                     <mesh filename="package://four_ws_robot_description/meshes/DAE/base/base.dae" />
                 </geometry>
-                <origin xyz="0.0 0.0 0.0" />
+                <origin xyz="0 0 0" />
             </visual>
             <collision>
@@ -18,9 +18,9 @@
                     <mesh filename="package://four_ws_robot_description/meshes/STL/base/base.stl" />
                 </geometry>
-                <origin xyz="0.0 0.0 0.0" />
+                <origin xyz="0 0 0" />
             </collision>
             <inertial>
                 <mass value="1.2" />
-                <origin xyz="0 0 0.017" />
+                <origin xyz="-0.002589 -0.000065 0.015452" />
                 <inertia ixx="0.0001873" ixy="0" ixz="0" iyy="0.000055" iyz="0" izz="0.0002283" />
             </inertial>

File: four_ws_robot_description/urdf/camera/camera.urdf.xacro (robot description, xacro)
@@ -12,5 +12,5 @@
                     <mesh filename="package://four_ws_robot_description/meshes/DAE/camera/camera.dae" />
                 </geometry>
-                <origin xyz="0.0 0.0 0.0" />
+                <origin xyz="0 0 0" />
             </visual>
             <collision>
@@ -18,9 +18,9 @@
                     <mesh filename="package://four_ws_robot_description/meshes/STL/camera/camera.stl" />
                 </geometry>
-                <origin xyz="0.0 0.0 0.0" />
+                <origin xyz="0 0 0" />
             </collision>
             <inertial>
                 <mass value="0.1" />
-                <origin xyz="0.0 0.0 0.0" />
+                <origin xyz="-0.005184 0 -0.000066" />
                 <inertia ixx="0.00001" ixy="0" ixz="0" iyy="0.00001" iyz="0" izz="0.00001" />
             </inertial>

File: four_ws_robot_description/urdf/lidar_base/lidar_base.urdf.xacro (robot description, xacro)
@@ -12,5 +12,5 @@
                     <mesh filename="package://four_ws_robot_description/meshes/DAE/lidar_base/YDlidar_base.dae" />
                 </geometry>
-                <origin xyz="0.0 0.0 0.0" />
+                <origin xyz="0 0 0" />
             </visual>
             <collision>
@@ -18,9 +18,9 @@
                     <mesh filename="package://four_ws_robot_description/meshes/STL/lidar_base/YDlidar_base.stl" />
                 </geometry>
-                <origin xyz="0.0 0.0 0.0" />
+                <origin xyz="0 0 0" />
             </collision>
             <inertial>
                 <mass value="0.2" />
-                <origin xyz="0.0 0.0 0.017" />
+                <origin xyz="0.042143 0 0.025917" />
                 <inertia ixx="0.0000873" ixy="0" ixz="0" iyy="0.000005" iyz="0" izz="0.0000283" />
             </inertial>

File: four_ws_robot_description/urdf/lidar_head/lidar_head.urdf.xacro (robot description, xacro)
@@ -12,5 +12,5 @@
                     <mesh filename="package://four_ws_robot_description/meshes/DAE/lidar_head/YDlidar_head.dae" />
                 </geometry>
-                <origin xyz="0.0 0.0 0.0" />
+                <origin xyz="0 0 0" />
             </visual>
             <collision>
@@ -18,9 +18,9 @@
                     <mesh filename="package://four_ws_robot_description/meshes/STL/lidar_head/YDlidar_head.stl" />
                 </geometry>
-                <origin xyz="0.0 0.0 0.0" />
+                <origin xyz="0 0 0" />
             </collision>
             <inertial>
                 <mass value="0.05" />
-                <origin xyz="0.0 0.0 0.0" />
+                <origin xyz="-0.00014 0.001365 0.048638" />
                 <inertia ixx="0.00001" ixy="0" ixz="0" iyy="0.000018" iyz="0" izz="0.00001" />
             </inertial>

File: four_ws_robot_description/urdf/steering/steering.urdf.xacro (robot description, xacro)
@@ -14,5 +14,5 @@
                     <mesh filename="package://four_ws_robot_description/meshes/DAE/steering/${prefix}_steering.dae" />
                 </geometry>
-                <origin xyz="0.0 0.0 0.0" />
+                <origin xyz="0 0 0" />
             </visual>
             <collision>
@@ -20,9 +20,9 @@
                     <mesh filename="package://four_ws_robot_description/meshes/STL/steering/steering.stl" />
                 </geometry>
-                <origin xyz="0.0 0.0 0.0" />
+                <origin xyz="0 0 0" />
             </collision>
             <inertial>
                 <mass value="0.15" />
-                <origin xyz="0.0 0.0 -0.02" />
+                <origin xyz="0 0 -0.02" />
                 <inertia ixx="0.00001" ixy="0" ixz="0" iyy="0.00001" iyz="0" izz="0.000004" />
             </inertial>

File: four_ws_robot_description/urdf/wheel/wheel.urdf.xacro (robot description, xacro)
@@ -14,5 +14,5 @@
                     <mesh filename="package://four_ws_robot_description/meshes/DAE/wheel/wheel.dae" />
                 </geometry>
-                <origin xyz="0.0 0.0 0.0" />
+                <origin xyz="0 0 0" />
             </visual>
             <collision>
@@ -20,9 +20,9 @@
                     <mesh filename="package://four_ws_robot_description/meshes/STL/wheel/wheel.stl" />
                 </geometry>
-                <origin xyz="0.0 0.0 0.0" />
+                <origin xyz="0 0 0" />
             </collision>
             <inertial>
                 <mass value="0.05" />
-                <origin xyz="0.0 -0.007 0.0" />
+                <origin xyz="0 -0.007685 0" />
                 <inertia ixx="0.00001" ixy="0" ixz="0" iyy="0.000018" iyz="0" izz="0.00001" />
             </inertial>
