Commit message: исправил опечатки с transmission описаниях подвески и колес + в описании робота

File: four_ws_robot_description/urdf/four_ws_robot.urdf.xacro (robot description, xacro)
@@ -33,5 +33,5 @@
         <origin xyz="0.022 0 0.0" rpy="0 0 0" />
     </xacro:lidar_head>
-    <xacro:lidar_head_gazebo min_rad="-${M_PI}" max_rad="${M_PI}" min_range="0.15" max_range="8" />
+    <xacro:lidar_head_gazebo min_angle="-${M_PI}" max_angle="${M_PI}" min_range="0.15" max_range="8" />
     <!-- camera -->
     <xacro:camera parent="base_link">

File: four_ws_robot_description/urdf/macros/lidar_head/lidar_head.gazebo.xacro (robot description, xacro)
@@ -1,5 +1,5 @@
 <?xml version="1.0"?>
 <robot xmlns:xacro="http://ros.org/wiki/xacro">
-    <xacro:macro name="lidar_head_gazebo" params="min_rad max_rad min_range max_range">
+    <xacro:macro name="lidar_head_gazebo" params="min_angle max_angle min_range max_range">
         <gazebo reference="lidar_head_link">
             <selfCollide>false</selfCollide>
@@ -15,6 +15,6 @@
                             <samples>360</samples>
                             <resolution>1</resolution>
-                            <min_angle>${min_rad}</min_angle>
-                            <max_angle>${max_rad}</max_angle>
+                            <min_angle>${min_angle}</min_angle>
+                            <max_angle>${max_angle}</max_angle>
                         </horizontal>
                     </scan>

File: four_ws_robot_description/urdf/macros/steering/steering.transmission.xacro (robot description, xacro)
@@ -5,8 +5,8 @@
             <type>transmission_interface/SimpleTransmission</type>
             <joint name="${prefix}_steering_joint">
-                <hardwareInterface>hardware_interface/PositionJointInterface</hardwareInterface>
+                <hardwareInterface>PositionJointInterface</hardwareInterface>
             </joint>
             <actuator name="${prefix}_steering_motor">
-                <hardwareInterface>hardware_interface/PositionJointInterface</hardwareInterface>
+                <hardwareInterface>PositionJointInterface</hardwareInterface>
                 <mechanicalReduction>30</mechanicalReduction>
             </actuator>

File: four_ws_robot_description/urdf/macros/wheel/wheel.transmission.xacro (robot description, xacro)
@@ -5,8 +5,8 @@
             <type>transmission_interface/SimpleTransmission</type>
             <joint name="${prefix}_wheel_joint">
-                <hardwareInterface>hardware_interface/VelocityJointInterface</hardwareInterface>
+                <hardwareInterface>VelocityJointInterface</hardwareInterface>
             </joint>
             <actuator name="${prefix}_wheel_motor">
-                <hardwareInterface>hardware_interface/VelocityJointInterface</hardwareInterface>
+                <hardwareInterface>VelocityJointInterface</hardwareInterface>
                 <mechanicalReduction>1</mechanicalReduction>
             </actuator>

Commit message: лаунч запуска контроллеров перенес в лаунч запуска симуляции, вернул hardware_interface в макрос описания трансмиссии колес и подвески, убрал переменную M_PI - будем использовать встроенную

File: four_ws_robot_description/urdf/four_ws_robot.urdf.xacro (robot description, xacro)
@@ -1,5 +1,4 @@
 <?xml version="1.0"?>
 <robot xmlns:xacro="http://ros.org/wiki/xacro" name="four_ws_robot">
-    <xacro:property name="M_PI" value="3.14159274" />
     <xacro:include filename="$(find four_ws_robot_description)/urdf/macros/base/base.urdf.xacro" />
     <xacro:include filename="$(find four_ws_robot_description)/urdf/macros/base/base.gazebo.xacro" />
@@ -33,5 +32,5 @@
         <origin xyz="0.022 0 0.0" rpy="0 0 0" />
     </xacro:lidar_head>
-    <xacro:lidar_head_gazebo min_angle="-${M_PI}" max_angle="${M_PI}" min_range="0.15" max_range="8" />
+    <xacro:lidar_head_gazebo min_angle="-${pi}" max_angle="${pi}" min_range="0.15" max_range="8" />
     <!-- camera -->
     <xacro:camera parent="base_link">
@@ -71,5 +70,5 @@
     <!-- front left -->
     <xacro:wheel prefix="front_left" parent="front_left_steering_link">
-        <origin xyz="0 0.021 -0.025" rpy="0 0 ${M_PI}" />
+        <origin xyz="0 0.021 -0.025" rpy="0 0 ${pi}" />
         <axis xyz="0 -1 0" />
     </xacro:wheel>
@@ -85,5 +84,5 @@
     <!--  rear left -->
     <xacro:wheel prefix="rear_left" parent="rear_left_steering_link">
-        <origin xyz="0 0.021 -0.025" rpy="0 0 ${M_PI}" />
+        <origin xyz="0 0.021 -0.025" rpy="0 0 ${pi}" />
         <axis xyz="0 -1 0" />
     </xacro:wheel>

File: four_ws_robot_description/urdf/macros/steering/steering.transmission.xacro (robot description, xacro)
@@ -5,8 +5,8 @@
             <type>transmission_interface/SimpleTransmission</type>
             <joint name="${prefix}_steering_joint">
-                <hardwareInterface>PositionJointInterface</hardwareInterface>
+                <hardwareInterface>hardware_interface/PositionJointInterface</hardwareInterface>
             </joint>
             <actuator name="${prefix}_steering_motor">
-                <hardwareInterface>PositionJointInterface</hardwareInterface>
+                <hardwareInterface>hardware_interface/PositionJointInterface</hardwareInterface>
                 <mechanicalReduction>30</mechanicalReduction>
             </actuator>

File: four_ws_robot_description/urdf/macros/wheel/wheel.transmission.xacro (robot description, xacro)
@@ -5,8 +5,8 @@
             <type>transmission_interface/SimpleTransmission</type>
             <joint name="${prefix}_wheel_joint">
-                <hardwareInterface>VelocityJointInterface</hardwareInterface>
+                <hardwareInterface>hardware_interface/VelocityJointInterface</hardwareInterface>
             </joint>
             <actuator name="${prefix}_wheel_motor">
-                <hardwareInterface>VelocityJointInterface</hardwareInterface>
+                <hardwareInterface>hardware_interface/VelocityJointInterface</hardwareInterface>
                 <mechanicalReduction>1</mechanicalReduction>
             </actuator>

Commit message: поменял описание передачи переменных как в ros_shared

File: four_ws_robot_description/urdf/four_ws_robot.urdf.xacro (robot description, xacro)
@@ -40,58 +40,74 @@
     <!-- steering -->
     <!-- front right -->
-    <xacro:steering prefix="front_right" parent="base_link">
-        <origin xyz="0.077 -0.031 -0.004" rpy="0 0 0" />
-        <axis xyz="0 0 1" />
-    </xacro:steering>
+    <xacro:steering
+        prefix="front_right"
+        parent="base_link"
+        origin_xyz="0.077 -0.031 -0.004"
+        origin_rpy="0 0 0"
+        axis_xyz="0 0 1" />
     <xacro:steering_gazebo prefix="front_right" />
     <xacro:steering_trans prefix="front_right" />
     <!-- front left -->
-    <xacro:steering prefix="front_left" parent="base_link">
-        <origin xyz="0.077 0.031 -0.004" rpy="0 0 0" />
-        <axis xyz="0 0 1" />
-    </xacro:steering>
+    <xacro:steering
+        prefix="front_left"
+        parent="base_link"
+        origin_xyz="0.077 0.031 -0.004"
+        origin_rpy="0 0 0"
+        axis_xyz="0 0 1" />
     <xacro:steering_gazebo prefix="front_left" />
     <xacro:steering_trans prefix="front_left" />
     <!-- rear right -->
-    <xacro:steering prefix="rear_right" parent="base_link">
-        <origin xyz="-0.077 -0.031 -0.004" rpy="0 0 0" />
-        <axis xyz="0 0 1" />
-    </xacro:steering>
+    <xacro:steering
+        prefix="rear_right"
+        parent="base_link"
+        origin_xyz="-0.077 -0.031 -0.004"
+        origin_rpy="0 0 0"
+        axis_xyz="0 0 1" />
     <xacro:steering_gazebo prefix="rear_right" />
     <xacro:steering_trans prefix="rear_right" />
     <!-- rear left -->
-    <xacro:steering prefix="rear_left" parent="base_link">
-        <origin xyz="-0.077 0.031 -0.004" rpy="0 0 0" />
-        <axis xyz="0 0 1" />
-    </xacro:steering>
+    <xacro:steering
+        prefix="rear_left"
+        parent="base_link"
+        origin_xyz="-0.077 0.031 -0.004"
+        origin_rpy="0 0 0"
+        axis_xyz="0 0 1" />
     <xacro:steering_gazebo prefix="rear_left" />
     <xacro:steering_trans prefix="rear_left" />
     <!-- wheel -->
     <!-- front left -->
-    <xacro:wheel prefix="front_left" parent="front_left_steering_link">
-        <origin xyz="0 0.021 -0.025" rpy="0 0 ${pi}" />
-        <axis xyz="0 -1 0" />
-    </xacro:wheel>
+    <xacro:wheel
+        prefix="front_left"
+        parent="front_left_steering_link"
+        origin_xyz="0 0.021 -0.025"
+        origin_rpy="0 0 ${pi}"
+        axis_xyz="0 -1 0" />
     <xacro:wheel_gazebo prefix="front_left" />
     <xacro:wheel_trans prefix="front_left" />
     <!-- front right -->
-    <xacro:wheel prefix="front_right" parent="front_right_steering_link">
-        <origin xyz="0 -0.021 -0.025" rpy="0 0 0" />
-        <axis xyz="0 1 0" />
-    </xacro:wheel>
+    <xacro:wheel
+        prefix="front_right"
+        parent="front_right_steering_link"
+        origin_xyz="0 -0.021 -0.025"
+        origin_rpy="0 0 0"
+        axis_xyz="0 1 0" />
     <xacro:wheel_gazebo prefix="front_right" />
     <xacro:wheel_trans prefix="front_right" />
     <!--  rear left -->
-    <xacro:wheel prefix="rear_left" parent="rear_left_steering_link">
-        <origin xyz="0 0.021 -0.025" rpy="0 0 ${pi}" />
-        <axis xyz="0 -1 0" />
-    </xacro:wheel>
+    <xacro:wheel
+        prefix="rear_left"
+        parent="rear_left_steering_link"
+        origin_xyz="0 0.021 -0.025"
+        origin_rpy="0 0 ${pi}"
+        axis_xyz="0 -1 0" />
     <xacro:wheel_gazebo prefix="rear_left" />
     <xacro:wheel_trans prefix="rear_left" />
     <!-- rear right -->
-    <xacro:wheel prefix="rear_right" parent="rear_right_steering_link">
-        <origin xyz="0 -0.021 -0.025" rpy="0 0 0" />
-        <axis xyz="0 1 0" />
-    </xacro:wheel>
+    <xacro:wheel
+        prefix="rear_right"
+        parent="rear_right_steering_link"
+        origin_xyz="0 -0.021 -0.025"
+        origin_rpy="0 0 0"
+        axis_xyz="0 1 0" />
     <xacro:wheel_gazebo prefix="rear_right" />
     <xacro:wheel_trans prefix="rear_right" />
@@ -106,5 +122,5 @@
         <!-- plugin that publishes the position of the coordinate system "bodyName"
         relative to "frameName" in the topic "ground_truth/state" -->
-        <plugin name="p3d_base_controller" filename="libgazebo_ros_p3d.so">
+        <plugin name="gazebo_ros_p3d" filename="libgazebo_ros_p3d.so">
             <alwaysOn>true</alwaysOn>
             <updateRate>10</updateRate>

File: four_ws_robot_description/urdf/macros/steering/steering.urdf.xacro (robot description, xacro)
@@ -1,10 +1,10 @@
 <?xml version="1.0"?>
 <robot xmlns:xacro="http://ros.org/wiki/xacro">
-    <xacro:macro name="steering" params="prefix parent *joint_origin *joint_axis">
+    <xacro:macro name="steering" params="prefix parent origin_xyz origin_rpy axis_xyz">
         <joint name="${prefix}_steering_joint" type="revolute">
             <parent link="${parent}" />
             <child link="${prefix}_steering_link" />
-            <xacro:insert_block name="joint_origin" />
-            <xacro:insert_block name="joint_axis" />
+            <origin xyz="${origin_xyz}" rpy="${origin_rpy}" />
+            <axis xyz="${axis_xyz}" />
             <limit effort="5" velocity="6.28" lower="-2.1" upper="2.1" />
         </joint>

File: four_ws_robot_description/urdf/macros/wheel/wheel.urdf.xacro (robot description, xacro)
@@ -1,10 +1,10 @@
 <?xml version="1.0"?>
 <robot xmlns:xacro="http://ros.org/wiki/xacro">
-    <xacro:macro name="wheel" params="prefix parent *joint_origin *joint_axis">
+    <xacro:macro name="wheel" params="prefix parent origin_xyz origin_rpy axis_xyz">
         <joint name="${prefix}_wheel_joint" type="continuous">
             <parent link="${parent}" />
             <child link="${prefix}_wheel_link" />
-            <xacro:insert_block name="joint_origin" />
-            <xacro:insert_block name="joint_axis" />
+            <origin xyz="${origin_xyz}" rpy="${origin_rpy}" />
+            <axis xyz="${axis_xyz}" />
             <limit effort="1.5" velocity="20" />
         </joint>

Commit message: добавил макрос для imu, добавил отображение в rviz; переписал некоторые макросы без использования макроса `insert_block`

File: four_ws_robot_description/urdf/four_ws_robot.urdf.xacro (robot description, xacro)
@@ -1,15 +1,24 @@
 <?xml version="1.0"?>
 <robot xmlns:xacro="http://ros.org/wiki/xacro" name="four_ws_robot">
+    <!-- base -->
     <xacro:include filename="$(find four_ws_robot_description)/urdf/macros/base/base.urdf.xacro" />
     <xacro:include filename="$(find four_ws_robot_description)/urdf/macros/base/base.gazebo.xacro" />
+    <!-- lidar_base -->
+    <xacro:include filename="$(find four_ws_robot_description)/urdf/macros/lidar_base/lidar_base.urdf.xacro" />
+    <xacro:include filename="$(find four_ws_robot_description)/urdf/macros/lidar_base/lidar_base.gazebo.xacro" />
+    <!-- lidar_head -->
+    <xacro:include filename="$(find four_ws_robot_description)/urdf/macros/lidar_head/lidar_head.urdf.xacro" />
+    <xacro:include filename="$(find four_ws_robot_description)/urdf/macros/lidar_head/lidar_head.gazebo.xacro" />
+    <!-- camera -->
     <xacro:include filename="$(find four_ws_robot_description)/urdf/macros/camera/camera.urdf.xacro" />
     <xacro:include filename="$(find four_ws_robot_description)/urdf/macros/camera/camera.gazebo.xacro" />
-    <xacro:include filename="$(find four_ws_robot_description)/urdf/macros/lidar_base/lidar_base.urdf.xacro" />
-    <xacro:include filename="$(find four_ws_robot_description)/urdf/macros/lidar_base/lidar_base.gazebo.xacro" />
-    <xacro:include filename="$(find four_ws_robot_description)/urdf/macros/lidar_head/lidar_head.urdf.xacro" />
-    <xacro:include filename="$(find four_ws_robot_description)/urdf/macros/lidar_head/lidar_head.gazebo.xacro" />
+    <!-- imu -->
+    <xacro:include filename="$(find four_ws_robot_description)/urdf/macros/imu/imu.urdf.xacro" />
+    <xacro:include filename="$(find four_ws_robot_description)/urdf/macros/imu/imu.gazebo.xacro" />
+    <!-- steering -->
     <xacro:include filename="$(find four_ws_robot_description)/urdf/macros/steering/steering.urdf.xacro" />
     <xacro:include filename="$(find four_ws_robot_description)/urdf/macros/steering/steering.gazebo.xacro" />
     <xacro:include filename="$(find four_ws_robot_description)/urdf/macros/steering/steering.transmission.xacro" />
+    <!-- wheels -->
     <xacro:include filename="$(find four_ws_robot_description)/urdf/macros/wheel/wheel.urdf.xacro" />
     <xacro:include filename="$(find four_ws_robot_description)/urdf/macros/wheel/wheel.gazebo.xacro" />
@@ -19,23 +28,33 @@
     <gazebo reference="base_footprint" />
     <!-- base -->
-    <xacro:base parent="base_footprint">
-        <origin xyz="0 0 0.055" rpy="0 0 0" />
-    </xacro:base>
+    <xacro:base
+        parent="base_footprint"
+        origin_xyz="0 0 0.055"
+        origin_rpy="0 0 0" />
     <xacro:base_gazebo />
     <!-- lidar_base -->
-    <xacro:lidar_base parent="base_link">
-        <origin xyz="-0.022 0 0.035" rpy="0 0 0" />
-    </xacro:lidar_base>
+    <xacro:lidar_base
+        parent="base_link"
+        origin_xyz="-0.022 0 0.035"
+        origin_rpy="0 0 0" />
     <xacro:lidar_base_gazebo />
     <!-- lidar_head -->
-    <xacro:lidar_head parent="lidar_base_link">
-        <origin xyz="0.022 0 0.0" rpy="0 0 0" />
-    </xacro:lidar_head>
+    <xacro:lidar_head
+        parent="lidar_base_link"
+        origin_xyz="0.022 0 0"
+        origin_rpy="0 0 0" />
     <xacro:lidar_head_gazebo min_angle="-${pi}" max_angle="${pi}" min_range="0.15" max_range="8" />
     <!-- camera -->
-    <xacro:camera parent="base_link">
-        <origin xyz="0.1 0 0.0177" rpy="0 0 0" />
-    </xacro:camera>
+    <xacro:camera
+        parent="base_link"
+        origin_xyz="0.1 0 0.0177"
+        origin_rpy="0 0 0" />
     <xacro:camera_gazebo />
+    <!-- imu -->
+    <xacro:imu
+        parent="base_link"
+        origin_xyz="0 0 0"
+        origin_rpy="0 0 0" />
+    <xacro:imu_gazebo />
     <!-- steering -->
     <!-- front right -->
@@ -75,5 +94,5 @@
     <xacro:steering_gazebo prefix="rear_left" />
     <xacro:steering_trans prefix="rear_left" />
-    <!-- wheel -->
+    <!-- wheels -->
     <!-- front left -->
     <xacro:wheel

File: four_ws_robot_description/urdf/macros/base/base.urdf.xacro (robot description, xacro)
@@ -1,9 +1,9 @@
 <?xml version="1.0"?>
 <robot xmlns:xacro="http://ros.org/wiki/xacro">
-    <xacro:macro name="base" params="parent *joint_origin">
+    <xacro:macro name="base" params="parent origin_xyz origin_rpy">
         <joint name="base_link_joint" type="fixed">
             <parent link="${parent}" />
             <child link="base_link" />
-            <xacro:insert_block name="joint_origin" />
+            <origin xyz="${origin_xyz}" rpy="${origin_rpy}" />
         </joint>
         <link name="base_link">

File: four_ws_robot_description/urdf/macros/camera/camera.urdf.xacro (robot description, xacro)
@@ -1,9 +1,9 @@
 <?xml version="1.0"?>
 <robot xmlns:xacro="http://ros.org/wiki/xacro">
-    <xacro:macro name="camera" params="parent *joint_origin">
+    <xacro:macro name="camera" params="parent origin_xyz origin_rpy">
         <joint name="camera_joint" type="fixed">
             <parent link="${parent}" />
             <child link="camera_link" />
-            <xacro:insert_block name="joint_origin" />
+            <origin xyz="${origin_xyz}" rpy="${origin_rpy}" />
         </joint>
         <link name="camera_link">

File: four_ws_robot_description/urdf/macros/lidar_base/lidar_base.urdf.xacro (robot description, xacro)
@@ -1,9 +1,9 @@
 <?xml version="1.0"?>
 <robot xmlns:xacro="http://ros.org/wiki/xacro">
-    <xacro:macro name="lidar_base" params="parent *joint_origin">
+    <xacro:macro name="lidar_base" params="parent origin_xyz origin_rpy">
         <joint name="lidar_base_joint" type="fixed">
             <parent link="${parent}" />
             <child link="lidar_base_link" />
-            <xacro:insert_block name="joint_origin" />
+            <origin xyz="${origin_xyz}" rpy="${origin_rpy}" />
         </joint>
         <link name="lidar_base_link">

File: four_ws_robot_description/urdf/macros/lidar_head/lidar_head.urdf.xacro (robot description, xacro)
@@ -1,9 +1,9 @@
 <?xml version="1.0"?>
 <robot xmlns:xacro="http://ros.org/wiki/xacro">
-    <xacro:macro name="lidar_head" params="parent *joint_origin">
+    <xacro:macro name="lidar_head" params="parent origin_xyz origin_rpy">
         <joint name="lidar_head_joint" type="fixed">
             <parent link="${parent}" />
             <child link="lidar_head_link" />
-            <xacro:insert_block name="joint_origin" />
+            <origin xyz="${origin_xyz}" rpy="${origin_rpy}" />
         </joint>
         <link name="lidar_head_link">
