Commit message: переименовал "steering" в "steer" в urdf-макросах для будущей интеграции с ros_shared

File: four_ws_robot_description/urdf/four_ws_robot.urdf.xacro (robot description, xacro)
@@ -16,8 +16,8 @@
     <xacro:include filename="$(find four_ws_robot_description)/urdf/macros/imu/imu.urdf.xacro" />
     <xacro:include filename="$(find four_ws_robot_description)/urdf/macros/imu/imu.gazebo.xacro" />
-    <!-- steering -->
-    <xacro:include filename="$(find four_ws_robot_description)/urdf/macros/steering/steering.urdf.xacro" />
-    <xacro:include filename="$(find four_ws_robot_description)/urdf/macros/steering/steering.gazebo.xacro" />
-    <xacro:include filename="$(find four_ws_robot_description)/urdf/macros/steering/steering.transmission.xacro" />
+    <!-- steer -->
+    <xacro:include filename="$(find four_ws_robot_description)/urdf/macros/steer/steer.urdf.xacro" />
+    <xacro:include filename="$(find four_ws_robot_description)/urdf/macros/steer/steer.gazebo.xacro" />
+    <xacro:include filename="$(find four_ws_robot_description)/urdf/macros/steer/steer.transmission.xacro" />
     <!-- wheels -->
     <xacro:include filename="$(find four_ws_robot_description)/urdf/macros/wheel/wheel.urdf.xacro" />
@@ -57,7 +57,7 @@
         origin_rpy="0 0 0" />
     <xacro:imu_gazebo />
-    <!-- steering -->
+    <!-- steer -->
     <!-- front right -->
-    <xacro:steering
+    <xacro:steer
         prefix="front_right"
         parent="base_link"
@@ -65,8 +65,8 @@
         origin_rpy="0 0 0"
         axis_xyz="0 0 1" />
-    <xacro:steering_gazebo prefix="front_right" />
-    <xacro:steering_trans prefix="front_right" />
+    <xacro:steer_gazebo prefix="front_right" />
+    <xacro:steer_trans prefix="front_right" />
     <!-- front left -->
-    <xacro:steering
+    <xacro:steer
         prefix="front_left"
         parent="base_link"
@@ -74,8 +74,8 @@
         origin_rpy="0 0 0"
         axis_xyz="0 0 1" />
-    <xacro:steering_gazebo prefix="front_left" />
-    <xacro:steering_trans prefix="front_left" />
+    <xacro:steer_gazebo prefix="front_left" />
+    <xacro:steer_trans prefix="front_left" />
     <!-- rear right -->
-    <xacro:steering
+    <xacro:steer
         prefix="rear_right"
         parent="base_link"
@@ -83,8 +83,8 @@
         origin_rpy="0 0 0"
         axis_xyz="0 0 1" />
-    <xacro:steering_gazebo prefix="rear_right" />
-    <xacro:steering_trans prefix="rear_right" />
+    <xacro:steer_gazebo prefix="rear_right" />
+    <xacro:steer_trans prefix="rear_right" />
     <!-- rear left -->
-    <xacro:steering
+    <xacro:steer
         prefix="rear_left"
         parent="base_link"
@@ -92,11 +92,11 @@
         origin_rpy="0 0 0"
         axis_xyz="0 0 1" />
-    <xacro:steering_gazebo prefix="rear_left" />
-    <xacro:steering_trans prefix="rear_left" />
+    <xacro:steer_gazebo prefix="rear_left" />
+    <xacro:steer_trans prefix="rear_left" />
     <!-- wheels -->
     <!-- front left -->
     <xacro:wheel
         prefix="front_left"
-        parent="front_left_steering_link"
+        parent="front_left_steer_link"
         origin_xyz="0 0.021 -0.025"
         origin_rpy="0 0 ${pi}"
@@ -107,5 +107,5 @@
     <xacro:wheel
         prefix="front_right"
-        parent="front_right_steering_link"
+        parent="front_right_steer_link"
         origin_xyz="0 -0.021 -0.025"
         origin_rpy="0 0 0"
@@ -116,5 +116,5 @@
     <xacro:wheel
         prefix="rear_left"
-        parent="rear_left_steering_link"
+        parent="rear_left_steer_link"
         origin_xyz="0 0.021 -0.025"
         origin_rpy="0 0 ${pi}"
@@ -125,5 +125,5 @@
     <xacro:wheel
         prefix="rear_right"
-        parent="rear_right_steering_link"
+        parent="rear_right_steer_link"
         origin_xyz="0 -0.021 -0.025"
         origin_rpy="0 0 0"
@@ -145,5 +145,5 @@
             <bodyName>base_footprint</bodyName>
             <topicName>ground_truth/state</topicName>
-            <frameName>world</frameName>
+            <frameName>map</frameName>
             <xyzOffsets>0 0 0</xyzOffsets>
             <rpyOffsets>0 0 0</rpyOffsets>

File: four_ws_robot_description/urdf/macros/imu/imu.urdf.xacro (robot description, xacro)
@@ -2,4 +2,5 @@
 <robot xmlns:xacro="http://www.ros.org/wiki/xacro">
     <xacro:include filename="$(find maddrive_urdf_tools)/urdf/macros/inertia.urdf.xacro" />
+    <xacro:include filename="$(find maddrive_urdf_tools)/urdf/macros/common.urdf.xacro" />
     <xacro:property name="rs_imu_height" value="0.01" />
     <xacro:property name="rs_imu_width" value="0.01" />
@@ -22,5 +23,5 @@
                 </geometry>
             </collision>
-            <xacro:null_inertial />
+            <xacro:null_inertia />
         </link>
     </xacro:macro>

File: four_ws_robot_description/urdf/macros/steer/steer.gazebo.xacro (robot description, xacro)
@@ -1,6 +1,6 @@
 <?xml version="1.0"?>
 <robot xmlns:xacro="http://ros.org/wiki/xacro">
-    <xacro:macro name="steering_gazebo" params="prefix">
-        <gazebo reference="${prefix}_steering_link">
+    <xacro:macro name="steer_gazebo" params="prefix">
+        <gazebo reference="${prefix}_steer_link">
             <selfCollide>false</selfCollide>
             <mu1 value="0.05" />

File: four_ws_robot_description/urdf/macros/steer/steer.transmission.xacro (robot description, xacro)
@@ -1,11 +1,11 @@
 <?xml version="1.0"?>
 <robot xmlns:xacro="http://ros.org/wiki/xacro">
-    <xacro:macro name="steering_trans" params="prefix">
-        <transmission name="${prefix}_steering_trans">
+    <xacro:macro name="steer_trans" params="prefix">
+        <transmission name="${prefix}_steer_trans">
             <type>transmission_interface/SimpleTransmission</type>
-            <joint name="${prefix}_steering_joint">
+            <joint name="${prefix}_steer_joint">
                 <hardwareInterface>hardware_interface/PositionJointInterface</hardwareInterface>
             </joint>
-            <actuator name="${prefix}_steering_motor">
+            <actuator name="${prefix}_steer_motor">
                 <hardwareInterface>hardware_interface/PositionJointInterface</hardwareInterface>
                 <mechanicalReduction>30</mechanicalReduction>

File: four_ws_robot_description/urdf/macros/steer/steer.urdf.xacro (robot description, xacro)
@@ -1,16 +1,16 @@
 <?xml version="1.0"?>
 <robot xmlns:xacro="http://ros.org/wiki/xacro">
-    <xacro:macro name="steering" params="prefix parent origin_xyz origin_rpy axis_xyz">
-        <joint name="${prefix}_steering_joint" type="revolute">
+    <xacro:macro name="steer" params="prefix parent origin_xyz origin_rpy axis_xyz">
+        <joint name="${prefix}_steer_joint" type="revolute">
             <parent link="${parent}" />
-            <child link="${prefix}_steering_link" />
+            <child link="${prefix}_steer_link" />
             <origin xyz="${origin_xyz}" rpy="${origin_rpy}" />
             <axis xyz="${axis_xyz}" />
             <limit effort="5" velocity="6.28" lower="-2.1" upper="2.1" />
         </joint>
-        <link name="${prefix}_steering_link">
+        <link name="${prefix}_steer_link">
             <visual>
                 <geometry>
-                    <mesh filename="package://four_ws_robot_description/meshes/DAE/steering/${prefix}_steering.dae" />
+                    <mesh filename="package://four_ws_robot_description/meshes/DAE/steer/${prefix}_steer.dae" />
                 </geometry>
                 <origin xyz="0 0 0" />
@@ -18,5 +18,5 @@
             <collision>
                 <geometry>
-                    <mesh filename="package://four_ws_robot_description/meshes/STL/steering/steering.stl" />
+                    <mesh filename="package://four_ws_robot_description/meshes/STL/steer/steer.stl" />
                 </geometry>
                 <origin xyz="0 0 0" />

Commit message: убрал отдельные макросы трансмиссии и газебо, все теперь находится в одном макросе

File: four_ws_robot_description/urdf/four_ws_robot.urdf.xacro (robot description, xacro)
@@ -3,25 +3,16 @@
     <!-- base -->
     <xacro:include filename="$(find four_ws_robot_description)/urdf/macros/base/base.urdf.xacro" />
-    <xacro:include filename="$(find four_ws_robot_description)/urdf/macros/base/base.gazebo.xacro" />
     <!-- lidar_base -->
     <xacro:include filename="$(find four_ws_robot_description)/urdf/macros/lidar_base/lidar_base.urdf.xacro" />
-    <xacro:include filename="$(find four_ws_robot_description)/urdf/macros/lidar_base/lidar_base.gazebo.xacro" />
     <!-- lidar_head -->
     <xacro:include filename="$(find four_ws_robot_description)/urdf/macros/lidar_head/lidar_head.urdf.xacro" />
-    <xacro:include filename="$(find four_ws_robot_description)/urdf/macros/lidar_head/lidar_head.gazebo.xacro" />
     <!-- camera -->
     <xacro:include filename="$(find four_ws_robot_description)/urdf/macros/camera/camera.urdf.xacro" />
-    <xacro:include filename="$(find four_ws_robot_description)/urdf/macros/camera/camera.gazebo.xacro" />
     <!-- imu -->
     <xacro:include filename="$(find four_ws_robot_description)/urdf/macros/imu/imu.urdf.xacro" />
-    <xacro:include filename="$(find four_ws_robot_description)/urdf/macros/imu/imu.gazebo.xacro" />
     <!-- steer -->
     <xacro:include filename="$(find four_ws_robot_description)/urdf/macros/steer/steer.urdf.xacro" />
-    <xacro:include filename="$(find four_ws_robot_description)/urdf/macros/steer/steer.gazebo.xacro" />
-    <xacro:include filename="$(find four_ws_robot_description)/urdf/macros/steer/steer.transmission.xacro" />
     <!-- wheels -->
     <xacro:include filename="$(find four_ws_robot_description)/urdf/macros/wheel/wheel.urdf.xacro" />
-    <xacro:include filename="$(find four_ws_robot_description)/urdf/macros/wheel/wheel.gazebo.xacro" />
-    <xacro:include filename="$(find four_ws_robot_description)/urdf/macros/wheel/wheel.transmission.xacro" />
     <!-- base_footprint -->
     <link name="base_footprint" />
@@ -32,5 +23,4 @@
         origin_xyz="0 0 0.055"
         origin_rpy="0 0 0" />
-    <xacro:base_gazebo />
     <!-- lidar_base -->
     <xacro:lidar_base
@@ -38,11 +28,13 @@
         origin_xyz="-0.022 0 0.035"
         origin_rpy="0 0 0" />
-    <xacro:lidar_base_gazebo />
     <!-- lidar_head -->
     <xacro:lidar_head
         parent="lidar_base_link"
         origin_xyz="0.022 0 0"
-        origin_rpy="0 0 0" />
-    <xacro:lidar_head_gazebo min_angle="-${pi}" max_angle="${pi}" min_range="0.15" max_range="8" />
+        origin_rpy="0 0 0"
+        min_angle="-${pi}"
+        max_angle="${pi}"
+        min_range="0.15"
+        max_range="8" />
     <!-- camera -->
     <xacro:camera
@@ -50,5 +42,4 @@
         origin_xyz="0.1 0 0.0177"
         origin_rpy="0 0 0" />
-    <xacro:camera_gazebo />
     <!-- imu -->
     <xacro:imu
@@ -56,5 +47,4 @@
         origin_xyz="0 0 0"
         origin_rpy="0 0 0" />
-    <xacro:imu_gazebo />
     <!-- steer -->
     <!-- front right -->
@@ -65,6 +55,4 @@
         origin_rpy="0 0 0"
         axis_xyz="0 0 1" />
-    <xacro:steer_gazebo prefix="front_right" />
-    <xacro:steer_trans prefix="front_right" />
     <!-- front left -->
     <xacro:steer
@@ -74,6 +62,4 @@
         origin_rpy="0 0 0"
         axis_xyz="0 0 1" />
-    <xacro:steer_gazebo prefix="front_left" />
-    <xacro:steer_trans prefix="front_left" />
     <!-- rear right -->
     <xacro:steer
@@ -83,6 +69,4 @@
         origin_rpy="0 0 0"
         axis_xyz="0 0 1" />
-    <xacro:steer_gazebo prefix="rear_right" />
-    <xacro:steer_trans prefix="rear_right" />
     <!-- rear left -->
     <xacro:steer
@@ -92,6 +76,4 @@
         origin_rpy="0 0 0"
         axis_xyz="0 0 1" />
-    <xacro:steer_gazebo prefix="rear_left" />
-    <xacro:steer_trans prefix="rear_left" />
     <!-- wheels -->
     <!-- front left -->
@@ -102,6 +84,4 @@
         origin_rpy="0 0 ${pi}"
         axis_xyz="0 -1 0" />
-    <xacro:wheel_gazebo prefix="front_left" />
-    <xacro:wheel_trans prefix="front_left" />
     <!-- front right -->
     <xacro:wheel
@@ -111,6 +91,4 @@
         origin_rpy="0 0 0"
         axis_xyz="0 1 0" />
-    <xacro:wheel_gazebo prefix="front_right" />
-    <xacro:wheel_trans prefix="front_right" />
     <!--  rear left -->
     <xacro:wheel
@@ -120,6 +98,4 @@
         origin_rpy="0 0 ${pi}"
         axis_xyz="0 -1 0" />
-    <xacro:wheel_gazebo prefix="rear_left" />
-    <xacro:wheel_trans prefix="rear_left" />
     <!-- rear right -->
     <xacro:wheel
@@ -129,6 +105,4 @@
         origin_rpy="0 0 0"
         axis_xyz="0 1 0" />
-    <xacro:wheel_gazebo prefix="rear_right" />
-    <xacro:wheel_trans prefix="rear_right" />
     <!-- gazebo plugins -->
     <gazebo>

File: four_ws_robot_description/urdf/macros/base/base.urdf.xacro (robot description, xacro)
@@ -26,4 +26,9 @@
             </inertial>
         </link>
+        <gazebo reference="base_link">
+            <selfCollide>false</selfCollide>
+            <mu1 value="0.05" />
+            <mu2 value="0.05" />
+        </gazebo>
     </xacro:macro>
 </robot>

File: four_ws_robot_description/urdf/macros/camera/camera.urdf.xacro (robot description, xacro)
@@ -26,4 +26,41 @@
             </inertial>
         </link>
+        <gazebo reference="camera_link">
+            <sensor name="camera" type="camera">
+                <pose>0 0 0 0 0 0</pose>
+                <visualize>true</visualize>
+                <update_rate>10</update_rate>
+                <camera>
+                    <horizontal_fov>1.3962634</horizontal_fov>
+                    <image>
+                        <format>R8G8B8</format>
+                        <width>640</width>
+                        <height>480</height>
+                    </image>
+                    <clip>
+                        <near>0.01</near>
+                        <far>100</far>
+                    </clip>
+                    <noise>
+                        <type>gaussian</type>
+                        <mean>0.0</mean>
+                        <stddev>0.01</stddev>
+                    </noise>
+                </camera>
+                <plugin name="camera_controller" filename="libgazebo_ros_camera.so">
+                    <updateRate>0.0</updateRate>
+                    <cameraName>camera</cameraName>
+                    <imageTopicName>image_raw</imageTopicName>
+                    <cameraInfoTopicName>camera_info</cameraInfoTopicName>
+                    <frameName>camera_link</frameName>
+                    <hackBaseline>0.07</hackBaseline>
+                    <distortionK1>0.0</distortionK1>
+                    <distortionK2>0.0</distortionK2>
+                    <distortionK3>0.0</distortionK3>
+                    <distortionT1>0.0</distortionT1>
+                    <distortionT2>0.0</distortionT2>
+                </plugin>
+            </sensor>
+        </gazebo>
     </xacro:macro>
 </robot>

File: four_ws_robot_description/urdf/macros/imu/imu.urdf.xacro (robot description, xacro)
@@ -25,4 +25,25 @@
             <xacro:null_inertia />
         </link>
+        <gazebo reference="imu_link">
+            <material>Gazebo/Red</material>
+            <gravity>true</gravity>
+            <sensor name="imu_sensor" type="imu">
+                <always_on>true</always_on>
+                <update_rate>100</update_rate>
+                <visualize>true</visualize>
+                <topic>__default_topic__</topic>
+                <plugin filename="libgazebo_ros_imu_sensor.so" name="imu_plugin">
+                    <topicName>/imu/</topicName>
+                    <bodyName>imu_link</bodyName>
+                    <updateRateHZ>20.0</updateRateHZ>
+                    <gaussianNoise>0.02</gaussianNoise>
+                    <xyzOffset>0 0 0</xyzOffset>
+                    <rpyOffset>0 0 0</rpyOffset>
+                    <frameName>imu_link</frameName>
+                    <initialOrientationAsReference>false</initialOrientationAsReference>
+                </plugin>
+                <pose>0 0 0 0 0 0</pose>
+            </sensor>
+        </gazebo>
     </xacro:macro>
 </robot>

File: four_ws_robot_description/urdf/macros/lidar_base/lidar_base.urdf.xacro (robot description, xacro)
@@ -26,4 +26,9 @@
             </inertial>
         </link>
+        <gazebo reference="lidar_base_link">
+            <selfCollide>false</selfCollide>
+            <mu1 value="0.05" />
+            <mu2 value="0.05" />
+        </gazebo>
     </xacro:macro>
 </robot>

File: four_ws_robot_description/urdf/macros/lidar_head/lidar_head.urdf.xacro (robot description, xacro)
@@ -1,5 +1,5 @@
 <?xml version="1.0"?>
 <robot xmlns:xacro="http://ros.org/wiki/xacro">
-    <xacro:macro name="lidar_head" params="parent origin_xyz origin_rpy">
+    <xacro:macro name="lidar_head" params="parent origin_xyz origin_rpy min_angle max_angle min_range max_range">
         <joint name="lidar_head_joint" type="fixed">
             <parent link="${parent}" />
@@ -26,4 +26,38 @@
             </inertial>
         </link>
+        <gazebo reference="lidar_head_link">
+            <selfCollide>false</selfCollide>
+            <mu1 value="0.05" />
+            <mu2 value="0.05" />
+            <sensor name="lidar_head_sensor" type="ray">
+                <pose>0 0 0.049 0 0 0</pose>
+                <visualize>true</visualize>
+                <update_rate>10</update_rate>
+                <ray>
+                    <scan>
+                        <horizontal>
+                            <samples>360</samples>
+                            <resolution>1</resolution>
+                            <min_angle>${min_angle}</min_angle>
+                            <max_angle>${max_angle}</max_angle>
+                        </horizontal>
+                    </scan>
+                    <range>
+                        <min>${min_range}</min>
+                        <max>${max_range}</max>
+                        <resolution>0.01</resolution>
+                    </range>
+                    <noise>
+                        <type>gaussian</type>
+                        <mean>0.0</mean>
+                        <stddev>0.03</stddev>
+                    </noise>
+                </ray>
+                <plugin name="gazebo_ros_lidar_head_controller" filename="libgazebo_ros_laser.so">
+                    <topicName>scan</topicName>
+                    <frameName>lidar_head_link</frameName>
+                </plugin>
+            </sensor>
+        </gazebo>
     </xacro:macro>
 </robot>

File: four_ws_robot_description/urdf/macros/steer/steer.urdf.xacro (robot description, xacro)
@@ -9,4 +9,14 @@
             <limit effort="5" velocity="6.28" lower="-2.1" upper="2.1" />
         </joint>
+        <transmission name="${prefix}_steer_trans">
+            <type>transmission_interface/SimpleTransmission</type>
+            <joint name="${prefix}_steer_joint">
+                <hardwareInterface>hardware_interface/PositionJointInterface</hardwareInterface>
+            </joint>
+            <actuator name="${prefix}_steer_motor">
+                <hardwareInterface>hardware_interface/PositionJointInterface</hardwareInterface>
+                <mechanicalReduction>30</mechanicalReduction>
+            </actuator>
+        </transmission>
         <link name="${prefix}_steer_link">
             <visual>
@@ -28,4 +38,9 @@
             </inertial>
         </link>
+        <gazebo reference="${prefix}_steer_link">
+            <selfCollide>false</selfCollide>
+            <mu1 value="0.05" />
+            <mu2 value="0.05" />
+        </gazebo>
     </xacro:macro>
 </robot>

File: four_ws_robot_description/urdf/macros/wheel/wheel.urdf.xacro (robot description, xacro)
@@ -9,4 +9,14 @@
             <limit effort="1.5" velocity="20" />
         </joint>
+        <transmission name="${prefix}_wheel_trans">
+            <type>transmission_interface/SimpleTransmission</type>
+            <joint name="${prefix}_wheel_joint">
+                <hardwareInterface>hardware_interface/VelocityJointInterface</hardwareInterface>
+            </joint>
+            <actuator name="${prefix}_wheel_motor">
+                <hardwareInterface>hardware_interface/VelocityJointInterface</hardwareInterface>
+                <mechanicalReduction>1</mechanicalReduction>
+            </actuator>
+        </transmission>
         <link name="${prefix}_wheel_link">
             <visual>
@@ -28,4 +38,9 @@
             </inertial>
         </link>
+        <gazebo reference="${prefix}_wheel_link">
+            <selfCollide>false</selfCollide>
+            <mu1 value="1.0" />
+            <mu2 value="1.0" />
+        </gazebo>
     </xacro:macro>
 </robot>
