Commit message: очередные неудачные попытки настроить ПИД (уменьшена масса робота); добавлено полное описание gazebo_ros_control

File: four_ws_robot_description/urdf/base.urdf.xacro (robot description, xacro)
@@ -94,5 +94,8 @@
 		<plugin name="gazebo_ros_control" filename="libgazebo_ros_control.so">
 			<robotNamespace>/</robotNamespace>
+			<robotParam>robot_description</robotParam>
 			<robotSimType>gazebo_ros_control/DefaultRobotHWSim</robotSimType>
+			<controlPeriod>0.01</controlPeriod>
+			<eStopTopic>gazebo_ros_control_stop</eStopTopic>
 		</plugin>
 		<!-- plugin that publishes the position of the coordinate system "bodyName"

File: four_ws_robot_description/urdf/params.urdf.xacro (robot description, xacro)
@@ -12,5 +12,5 @@
     <xacro:property name="body_width" value="0.8" />
     <xacro:property name="body_heigth" value="0.8" />
-    <xacro:property name="body_mass" value="40" />
+    <xacro:property name="body_mass" value="4" />
     <!-- габариты колес -->
     <xacro:property name="wheel_width" value="0.025" />
