Commit message: увеличил толщину "бампера" чтобы робот не переворачивался при столкновении

File: four_ws_robot_description/urdf/params.urdf.xacro (robot description, xacro)
@@ -4,6 +4,6 @@
     <xacro:property name="yaml_file" value="$(find four_ws_robot_description)/config/props.yaml" />
     <xacro:property name="props" value="${xacro.load_yaml(yaml_file)}" />
-    <xacro:property name="front_wheel_2_front_bumper" value="0.05" />
-    <xacro:property name="rear_wheel_2_rear_bumper" value="0.05" />
+    <xacro:property name="front_wheel_2_front_bumper" value="0.1" />
+    <xacro:property name="rear_wheel_2_rear_bumper" value="0.1" />
     <xacro:property name="wheelbase" value="${props['wheelbase']}" />
     <xacro:property name="track_width" value="${props['track_width']}" />

Commit message: подкорректировал ковариационные матрицы согласно отклонению сигнала GPS

File: four_ws_robot_description/urdf/params.urdf.xacro (robot description, xacro)
@@ -12,5 +12,5 @@
     <xacro:property name="body_width" value="0.8" />
     <xacro:property name="body_heigth" value="0.8" />
-    <xacro:property name="body_mass" value="4" />
+    <xacro:property name="body_mass" value="0.1" />
     <!-- габариты колес -->
     <xacro:property name="wheel_width" value="0.025" />
